File: tgs2611-c00.sch (EAGLE design)
At the start: 14 parts, among them J1 3.5mm, J2 M20-9980346, J3 TGS2611-C00, U1 INA219BIDCNT

Commit message: methane PCBs added
Parts:
- removed J1: 3.5mm, microbuilder:TERMBLOCK_1X2_3.5MM
- added R1: 10K, microbuilder:RESISTOR0603
- added U$1, U$6, U$7, U$8: MOUNTINGHOLE2.5, microbuilder:MOUNTINGHOLE2.5
- C1: device microbuilder:CAP_CERAMIC0603_NO -> microbuilder:CAP_CERAMIC0603
- C2: device microbuilder:CAP_CERAMIC0805-NOOUTLINE -> microbuilder:CAP_CERAMIC_0805MP
- R7: device microbuilder:RESISTOR_0603_NOOUT -> microbuilder:RESISTOR_0603MP
Connections:
- net GND: now also C1.P$2, C2.P$2, J2.1, J3.VH@2, R1.2; no longer C1.2, C2.2
- net SCL: now also J2.4
- net SDA: now also J2.3
- net VCC: now also C1.P$1, C2.P$1, J2.2, J3.VC+, J3.VH@1; no longer C1.1, C2.1
- net VIN+: now also J3.VC-, R1.1; no longer J1.2
- net VIN-: no longer J1.1
Other:
- moved on the sheet: C2, CONN3G$1, CONN4G$1, J2, J3
