File: Dream_leov1.kicad_sch (KiCad schematic)
At the start: 39 parts, among them IC1 TGS2611-C00, J1 GPIO, J11 10132328-10011LF, J2 Qwiic_Vertical, J3 679305124022, J4 Qwiic_Vertical, J5 M20-7830542, J6 Qwiic_Vertical, J7 5013310607, J8 Qwiic_4pin_Vertical, Q1 BSS138, U1 AP2112K-3.3, U2 BME280, U3 INA219BxDCN, U4 BME280, j9 Qwiic_Vertical

Commit message: halfway done v3
Parts:
- JP1, JP2, JP3, JP4: value ~ -> (none)
Connections:
- net GPIO18/PCM.CLK: now also R8.2
Other:
- moved on the sheet: D1, R8

Commit message: fixed issues; update schematic
Parts:
- removed R4: R_US, Resistor_SMD:R_0805_2012Metric, symbol Device:R_US
- removed U4: BME280, Package_LGA:Bosch_LGA-8_2.5x2.5mm_P0.65mm_ClockwisePinNumbering, symbol dk_Humidity-Moisture-Sensors:BME280
- added Q2: BSS138, SparkFun-Semiconductor-Standard:SOT-363, symbol SparkFun-DiscreteSemi:Q_NMOS_0.2A_50V_DUAL
- added R11, R12: 3.3k, Resistor_SMD:R_0402_1005Metric, symbol Device:R_US
- added R13: 10k, SparkFun-Resistor:R_Array_Convex_4x0603, symbol SparkFun-Resistor:10k_4x0603_Array
- added R4: PT2512FK-070R1L, downloaded:PT2512FK-070R1L, symbol PT2512FK-070R1L:PT2512FK-070R1L
- added U5: BME280, Package_LGA:Bosch_LGA-8_2.5x2.5mm_P0.65mm_ClockwisePinNumbering, symbol Sensor:BME280
- renumbered j9 to J9
Connections:
- net +5V: now also R11.1, R12.1; no longer J8.3 (Pin_3)
- net GND: now also J8.1 (Pin_1), U5.1 (GND), U5.7 (GND); no longer J8.4 (Pin_4)
- net GPIO22/SCL3: now also J9.4 (Pin_4); no longer J4.4 (Pin_4)
- net GPIO23/SDA4: now also J8.3 (Pin_3); no longer J8.2 (Pin_2)
- net GPIO24/SCL4: now also J8.4 (Pin_4); no longer J8.1 (Pin_1)
- net GPIO27/SDA3: now also J9.3 (Pin_3); no longer J4.3 (Pin_3)
- net GPIO2/SDA1: now also J2.3 (Pin_3), R12.2; no longer J9.3 (Pin_3)
- net GPIO3/SCL1: now also J2.4 (Pin_4), R11.2; no longer J9.4 (Pin_4)
- net GPIO5/SDA5: now also J4.3 (Pin_3), Q2.3 (D), R13.3; no longer J2.3 (Pin_3)
- net GPIO6/SCL5: now also J4.4 (Pin_4), Q2.6 (D), R13.1; no longer J2.4 (Pin_4)
- net INA+: now also R4.1
- net at U3.2 (IN-): now also R4.2
- net +3.3V renamed BME_3V3
- net BME_3V3: now also Q2.2 (G), Q2.5 (G), R13.6, R13.7, U5.2 (CSB), U5.6 (VDDIO), U5.8 (VDD); no longer C2.1, J1.1 (Pin_1), J1.17 (Pin_17), J2.2 (Pin_2), J5.3, J6.2 (Pin_2), J9.2 (Pin_2), R1.2, R1.4, U1.1 (VIN), U1.3 (EN)
- net BME_ADD renamed BME_ADD_1
- net BME_ADD_1: now also U5.5 (SDO); no longer U2.5 (SDO)
- net BME_SCL renamed BME_SCL1
- net BME_SCL1: now also U5.4 (SCK); no longer U2.4 (SCK)
- net BME_SDA renamed BME_SDA1
- net BME_SDA1: now also U5.3 (SDI); no longer U2.3 (SDI)
- new net +3V3: C2.1, J1.1 (Pin_1), J1.17 (Pin_17), J2.2 (Pin_2), J5.3, J6.2 (Pin_2), J8.2 (Pin_2), J9.2 (Pin_2), R1.2, R1.4, R13.2, R13.4, U1.1 (VIN), U1.3 (EN)
- new net BME_ADD_2: U2.5 (SDO)
- new net BME_SCL2: Q2.1 (S), R13.5, U2.4 (SCK)
- new net BME_SDA2: Q2.4 (S), R13.8, U2.3 (SDI)
Other:
- note added: "BME 280 - 1"
- note added: "BME 280 - 2"
- note added: "BME I2C Pullups"
- note added: "I2C BUS 1 QWIIC"
- note added: "I2C BUS 3 QWIIC"
- note added: "I2C BUS 4 QWIIC"
- note added: "I2C BUS 5 QWIIC"
- note added: "IPS7100 I2C QWIIC"
- note added: "Raspberry Pi Zero"
- note added: "TGS2611 METHANE SENSOR"
- note added: "UART QWIIC"
- note added: "USB-C POWER"
- note removed: "BME 280"
- note removed: "I2c Bus 4"
- note removed: "IPS7100"
- note removed: "QWIIC Connector - I2C Bus 1"
- note removed: "QWIIC Connector - I2C Bus 3"
- note removed: "QWIIC Connector - I2C Bus 5"
- note removed: "QWIIC Connector - UART"
- note removed: "Rasbery Pi Zero"
- note removed: "TGS2611_INA219"
- note removed: "usb-c power"
- company: (none) -> MINTS-AI Laboratory
- title: (none) -> DREAM
- moved on the sheet: C1, C2, C3, C4, C5, C6, C7, J2, J3, J4, J5, J6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
