File: methaneSensing/INIR2-ME5Mount.brd (EAGLE design)
At the start: 24 x 39 mm, 6 parts, among them J1 450-3326-01-03-00, J2 450-3326-01-03-00, J3 450-3326-01-03-00, J4 450-3326-01-03-00, J5 450-3326-01-03-00, J6 M20-9980346

Commit message: methane PCBs added
Parts:
- added U$1, U$2, U$3, U$4: MOUNTINGHOLE2.5, microbuilder:MOUNTINGHOLE_2.5_PLATED
Routing:
- net TX: track 41.9 -> 40.8 mm
- net 5V: track 64.8 -> 63.7 mm
Changed lines of the file:
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@@
 <wire x1="25" y1="37" x2="1" y2="37" width="0.2032" layer="20"/>
 <wire x1="1" y1="37" x2="1" y2="-2" width="0.2032" layer="20"/>
-<hole x="3" y="35" drill="0.35"/>
-<hole x="23" y="35" drill="0.35"/>
-<hole x="23" y="0" drill="0.35"/>
-<hole x="3" y="0" drill="0.35"/>
 </plain>
 <attributes>
@@
 <attribute name="VALUE" x="17.77" y="11.25" size="1.27" layer="27" rot="R180"/>
 </element>
+<element name="U$1" library="microbuilder" package="MOUNTINGHOLE_2.5_PLATED" value="MOUNTINGHOLE2.5" x="4" y="1" smashed="yes"/>
+<element name="U$2" library="microbuilder" package="MOUNTINGHOLE_2.5_PLATED" value="MOUNTINGHOLE2.5" x="22" y="1" smashed="yes"/>
+<element name="U$3" library="microbuilder" package="MOUNTINGHOLE_2.5_PLATED" value="MOUNTINGHOLE2.5" x="4" y="34" smashed="yes"/>
+<element name="U$4" library="microbuilder" package="MOUNTINGHOLE_2.5_PLATED" value="MOUNTINGHOLE2.5" x="22" y="34" smashed="yes"/>
 </elements>
 <signals>
@@
 <wire x1="18" y1="34" x2="9" y2="34" width="0.6059" layer="16"/>
 <wire x1="9" y1="34" x2="5" y2="30" width="0.6059" layer="16"/>
-<wire x1="5" y1="30" x2="5" y2="3" width="0.6059" layer="16"/>
-<wire x1="5" y1="3" x2="7" y2="1" width="0.6059" layer="16"/>
-<wire x1="14" y1="1" x2="7" y2="1" width="0.6059" layer="16"/>
+<wire x1="5" y1="30" x2="5" y2="5" width="0.6059" layer="16"/>
+<wire x1="5" y1="5" x2="9" y2="1" width="0.6059" layer="16"/>
+<wire x1="14" y1="1" x2="9" y2="1" width="0.6059" layer="16"/>
 <wire x1="16.54" y1="5.73" x2="14" y2="1" width="0.6059" layer="16"/>
 </signal>
@@
 <wire x1="11" y1="32" x2="13.335" y2="32" width="0.6059" layer="16"/>
 <wire x1="14" y1="5.73" x2="12.421965625" y2="3" width="0.6059" layer="16"/>
-<wire x1="12.421965625" y1="3" x2="9" y2="3" width="0.6059" layer="16"/>
-<wire x1="9" y1="3" x2="8" y2="4" width="0.6059" layer="16"/>
-<wire x1="8" y1="4" x2="8" y2="29" width="0.6059" layer="16"/>
+<wire x1="12.421965625" y1="3" x2="11" y2="3" width="0.6059" layer="16"/>
+<wire x1="11" y1="3" x2="8" y2="6" width="0.6059" layer="16"/>
+<wire x1="8" y1="6" x2="8" y2="29" width="0.6059" layer="16"/>
 <wire x1="8" y1="29" x2="11" y2="32" width="0.6059" layer="16"/>
 </signal>
