File: methaneSensing/SJH-5XDMount.sch.brd (EAGLE design)
At the start: 24 x 39 mm, 6 parts, among them J1 450-3326-01-03-00, J2 450-3326-01-03-00, J3 450-3326-01-03-00, J4 450-3326-01-03-00, J5 450-3326-01-03-00, J6 M20-9980346

Commit message: methane PCBs added
Parts:
- added U$1, U$2, U$3, U$4: MOUNTINGHOLE2.5, microbuilder:MOUNTINGHOLE_2.5_PLATED
Changed lines of the file:
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@@
 <wire x1="22" y1="42" x2="-2" y2="42" width="0.2032" layer="20"/>
 <wire x1="-2" y1="42" x2="-2" y2="3" width="0.2032" layer="20"/>
-<hole x="0" y="40" drill="0.35"/>
-<hole x="20" y="5" drill="0.35"/>
-<hole x="0" y="5" drill="0.35"/>
-<hole x="20" y="40" drill="0.35"/>
 </plain>
 <attributes>
@@
 <attribute name="VALUE" x="4.25" y="7.23" size="1.27" layer="27" rot="R90"/>
 </element>
+<element name="U$1" library="microbuilder" package="MOUNTINGHOLE_2.5_PLATED" value="MOUNTINGHOLE2.5" x="1" y="6" smashed="yes"/>
+<element name="U$2" library="microbuilder" package="MOUNTINGHOLE_2.5_PLATED" value="MOUNTINGHOLE2.5" x="19" y="6" smashed="yes"/>
+<element name="U$3" library="microbuilder" package="MOUNTINGHOLE_2.5_PLATED" value="MOUNTINGHOLE2.5" x="1" y="39" smashed="yes"/>
+<element name="U$4" library="microbuilder" package="MOUNTINGHOLE_2.5_PLATED" value="MOUNTINGHOLE2.5" x="19" y="39" smashed="yes"/>
 </elements>
 <signals>
