File: methaneSensing/SJH-5XDMount.sch.sch (EAGLE design)
At the start: 6 parts, among them J1 450-3326-01-03-00, J2 450-3326-01-03-00, J3 450-3326-01-03-00, J4 450-3326-01-03-00, J5 450-3326-01-03-00, J6 M20-9980346

Commit message: methane PCBs added
Parts:
- added U$1, U$2, U$3, U$4: MOUNTINGHOLE2.5, microbuilder:MOUNTINGHOLE2.5
Changed lines of the file:
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@@
 <part name="GND1" library="SparkFun-PowerSymbols" library_urn="urn:adsk.eagle:library:530" deviceset="GND" device=""/>
 <part name="SUPPLY1" library="SparkFun-PowerSymbols" library_urn="urn:adsk.eagle:library:530" deviceset="5V" device=""/>
+<part name="U$1" library="microbuilder" deviceset="MOUNTINGHOLE" device="2.5"/>
+<part name="U$2" library="microbuilder" deviceset="MOUNTINGHOLE" device="2.5"/>
+<part name="U$3" library="microbuilder" deviceset="MOUNTINGHOLE" device="2.5"/>
+<part name="U$4" library="microbuilder" deviceset="MOUNTINGHOLE" device="2.5"/>
 </parts>
 <sheets>
@@
 <attribute name="VALUE" x="-76.2" y="137.414" size="1.778" layer="96" font="vector" align="bottom-center"/>
 </instance>
+<instance part="U$1" gate="G$1" x="-170.18" y="142.24" smashed="yes"/>
+<instance part="U$2" gate="G$1" x="-162.56" y="142.24" smashed="yes"/>
+<instance part="U$3" gate="G$1" x="-149.86" y="142.24" smashed="yes"/>
+<instance part="U$4" gate="G$1" x="-142.24" y="142.24" smashed="yes"/>
 </instances>
 <busses>
