File: kiCad/dreamV1_0/dreamV1_0.kicad_pcb (KiCad board)
At the start: 2 copper layers, 80 x 80 mm, 35 parts, among them IC1 TGS2611-C00, J1 GPIO, J10 10132328-10011LF, J2 Qwiic_Vertical, J3 679305124022, J4 Qwiic_Vertical, J5 M20-7830542, J6 Qwiic_Vertical, J7 5013310607, J8 Qwiic_Vertical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

Commit message: PCB updates for dream
Parts:
- moved J2 79.5 mm to (68.0, 121.0), turned to 180 degrees
- moved J6 73.5 mm to (54.0, 71.0), turned to 180 degrees
- moved J4 53.0 mm to (118.2, 121.0), turned to 180 degrees
- moved J8 52.7 mm to (96.0, 104.0), turned to 180 degrees
- moved J7 46.4 mm to (87.0, 102.6)
- moved J9 20.2 mm to (126.0, 71.0), turned to 180 degrees
- moved C6 12.0 mm to (96.0, 84.3)
- moved C3 10.2 mm to (74.0, 122.0)
- moved R2 9.80 mm to (78.0, 117.0)
- moved C2 9.43 mm to (71.0, 112.0)
- moved C1 9.30 mm to (74.0, 117.0)
- moved U2 8.25 mm to (78.0, 122.0)
- moved R8 7.41 mm to (90.0, 89.0), turned to 0 degrees
- moved R4 6.32 mm to (88.0, 110.0)
- moved R5 6.20 mm to (123.0, 110.0)
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Other:
- board text added: "BME280"
- board text added: "INA219"

Commit message: PCB updates for dream
Parts:
- removed J10: 10132328-10011LF, downloaded:10132328-10011LF
- added J11: 10132328-10011LF, downloaded:10132328-10011LF, B.Cu at (90.0, 100.0)
- R6, R7: moved to B.Cu
- moved R7 55.0 mm to (84.0, 100.0), turned to 90 degrees
- moved R6 42.9 mm to (96.0, 100.0), turned to -90 degrees
- moved C2 10.5 mm to (74.0, 122.0)
- moved C1 10.0 mm to (74.0, 127.0), turned to 90 degrees
- moved R2 8.00 mm to (70.0, 117.0)
- moved J7 6.49 mm to (86.0, 109.0), turned to 0 degrees
- moved R8 6.00 mm to (90.0, 95.0)
- moved D1 5.53 mm to (90.0, 90.0)
- moved C7 5.52 mm to (90.0, 83.0)
- moved C4 5.00 mm to (103.0, 115.0)
- moved C5 5.00 mm to (114.1, 115.0)
- moved IC1 5.00 mm to (91.8, 125.0)
- moved J1 5.00 mm to (65.9, 77.0)
- moved J2 5.00 mm to (68.0, 126.0)
- moved J3 5.00 mm to (106.0, 126.5)
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Connections:
- R6 pad 1: Net-(J10-CC2) -> GND
- R6 pad 2: GND -> Net-(J11-CC2)
- R7 pad 1: Net-(J10-CC1) -> GND
- R7 pad 2: GND -> Net-(J11-CC1)
Other:
- outline, holes or cut-outs redrawn

Commit message: PCB updates for dream
Parts:
- added REF**: KiCad-Logo2_5mm_SilkScreen, Symbol:KiCad-Logo2_5mm_SilkScreen, F.Cu at (122.0, 58.0)
- added REF**: OSHW-Logo_5.7x6mm_SilkScreen, Symbol:OSHW-Logo_5.7x6mm_SilkScreen, F.Cu at (126.0, 65.0)
- R6, R7: footprint downloaded:RC0603N_YAG -> downloaded:RC0603N_YAG-L
- moved J7 40.7 mm to (90.0, 68.5)
- moved R6 12.0 mm to (84.0, 101.0), turned to 90 degrees
- moved R7 12.0 mm to (96.0, 101.0), turned to -90 degrees
- moved R8 7.26 mm to (95.0, 89.7), turned to 90 degrees
- moved J4 0.18 mm to (118.0, 126.0)
- turned C4 to -90 degrees
- turned C5 to -90 degrees
- turned C6 to 90 degrees
- turned JP3 to 90 degrees
Connections:
- J4 pad 4: /GPIO6/SCL5 -> /GPIO22/SCL3
Routing:
- net GND: track 0.00 -> 413.1 mm, vias 0 -> 5
- net +5V: track 0.00 -> 210.8 mm, vias 0 -> 6
- net +3V3: track 0.00 -> 167.7 mm, vias 0 -> 1
- net /GPIO23/SDA4: track 0.00 -> 100.9 mm, vias 0 -> 6
- net /GPIO27/SDA3: track 0.00 -> 98.3 mm, vias 0 -> 2
- net /GPIO24/SCL4: track 0.00 -> 96.9 mm, vias 0 -> 5
- net /GPIO6/SCL5: track 0.00 -> 96.2 mm, vias 0 -> 3
- net /GPIO22/SCL3: track 0.00 -> 96.1 mm, vias 0 -> 2
- net /GPIO2/SDA1: track 0.00 -> 93.2 mm, vias 0 -> 3
- net /GPIO3/SCL1: track 0.00 -> 90.2 mm, vias 0 -> 3
- net /GPIO5/SDA5: track 0.00 -> 83.7 mm, vias 0 -> 2
- net /5V_BUS_USB: track 0.00 -> 73.1 mm, vias 0 -> 1
- net /GPIO15/RXD0: track 0.00 -> 56.0 mm, vias 0 -> 1
- net BME_3V3: track 0.00 -> 55.4 mm
- net /GPIO14/TXD0: track 0.00 -> 49.3 mm
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Other:
- outline, holes or cut-outs redrawn
- board text added: "."
- board text added: "5v"
- board text added: "A0"
- board text added: "A1"
- board text added: "GND"
- board text added: "I2C Bus 1"
- board text added: "I2C Bus 3"
- board text added: "I2C Bus 4"
- board text added: "I2C Bus 5"
- board text added: "MINTS-AI Dream V1.0"
- board text added: "SPI"
- board text added: "UART"

Commit message: PCB updates for dream
Routing:
- net GND: track 413.1 -> 355.2 mm
- added copper zone on B.Cu, net GND
Changed lines of the file:
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@@
 		(model "${DIGIKEY_DOWNLOADED}/AB11AH-FC.step"
 			(offset
-				(xyz -2.25 0.25 -4)
+				(xyz -2.25 0.25 -3.5)
 			)
 			(scale
@@
 		)
 		(embedded_fonts no)
-		(model "TGS2611-C00.stp"
+		(model "${DIGIKEY_DOWNLOADED}/TGS2611-C00.stp"
 			(offset
 				(xyz 0 0 0)
@@
 		)
 		(embedded_fonts no)
+		(model "${DIGIKEY_DOWNLOADED}/RC0603N_YAG.step"
+			(offset
+				(xyz 0 0 0)
+			)
+			(scale
+				(xyz 1 1 1)
+			)
+			(rotate
+				(xyz 0 0 0)
+			)
+		)
 	)
 	(footprint "downloaded:RC0603N_YAG-L"
@@
 		)
 		(embedded_fonts no)
+		(model "${DIGIKEY_DOWNLOADED}/RC0603N_YAG.step"
+			(offset
+				(xyz 0 0 0)
+			)
+			(scale
+				(xyz 1 1 1)
+			)
+			(rotate
+				(xyz 0 0 0)
+			)
+		)
 	)
 	(footprint "downloaded:10132328-10011LF"
@@
 	)
 	(segment
-		(start 74.721 75.661)
-		(end 76.06 77)
-		(width 0.1)
-		(layer "F.Cu")
-		(net 1)
-	)
-	(segment
 		(start 98.822 113.3)
 		(end 97.5 111.978)
@@
 	)
 	(segment
-		(start 81.14 70.672)
-		(end 80.95 70.482)
-		(width 0.2)
-		(layer "F.Cu")
-		(net 1)
-	)
-	(segment
 		(start 84.76 81.712)
 		(end 85.014 81.458)
@@
 	)
 	(segment
-		(start 70.98 74.46)
-		(end 72.181 75.661)
-		(width 0.1)
-		(layer "F.Cu")
-		(net 1)
-	)
-	(segment
 		(start 126.416 113.716)
 		(end 126.416 112.954)
@@
 	)
 	(segment
-		(start 80.95 70.482)
-		(end 87.5 70.482)
-		(width 0.3)
-		(layer "F.Cu")
-		(net 1)
-	)
-	(segment
 		(start 77.5936 116.165)
 		(end 78.0106 115.748)
@@
 	)
 	(segment
-		(start 72.181 75.661)
-		(end 74.721 75.661)
-		(width 0.1)
-		(layer "F.Cu")
-		(net 1)
-	)
-	(segment
 		(start 119.5 124.489)
 		(end 119.5 119.0975)
@@
 	)
 	(segment
-		(start 70.98 74.46)
-		(end 74.958 70.482)
-		(width 0.3)
-		(layer "F.Cu")
-		(net 1)
-	)
-	(segment
 		(start 119.5 119.0975)
 		(end 118.1825 117.78)
@@
 	)
 	(segment
-		(start 74.958 70.482)
-		(end 80.95 70.482)
-		(width 0.3)
-		(layer "F.Cu")
-		(net 1)
-	)
-	(segment
 		(start 101.016 111.43)
 		(end 97.5 111.43)
@@
 	)
 	(segment
-		(start 81.14 74.46)
-		(end 81.14 70.672)
-		(width 0.2)
-		(layer "F.Cu")
-		(net 1)
-	)
-	(segment
 		(start 95.48895 83)
 		(end 96 83.51105)
@@
 	)
 	(segment
-		(start 100.071 75.849)
-		(end 101.46 74.46)
-		(width 0.2)
-		(layer "B.Cu")
-		(net 1)
-	)
-	(segment
 		(start 93.77 99)
 		(end 94.21 99.44)
@@
 	)
 	(segment
-		(start 97.531 75.849)
-		(end 100.071 75.849)
-		(width 0.2)
-		(layer "B.Cu")
-		(net 1)
-	)
-	(segment
 		(start 114.16 77)
 		(end 115.824 78.664)
@@
 	)
 	(segment
-		(start 106.54 74.46)
-		(end 107.929 75.849)
-		(width 0.2)
-		(layer "B.Cu")
-		(net 1)
-	)
-	(segment
 		(start 87.25 100.83)
 		(end 86.4 100.83)
@@
 	)
 	(segment
-		(start 94.996 75.616)
-		(end 96.38 77)
-		(width 0.2)
-		(layer "B.Cu")
-		(net 1)
-	)
-	(segment
-		(start 89.916 75.616)
-		(end 94.996 75.616)
-		(width 0.2)
-		(layer "B.Cu")
-		(net 1)
-	)
-	(segment
-		(start 101.46 74.46)
-		(end 102.611 73.309)
-		(width 0.2)
-		(layer "B.Cu")
-		(net 1)
-	)
-	(segment
 		(start 93.77 99)
 		(end 93.55 99)
@@
 	)
 	(segment
-		(start 102.611 73.309)
-		(end 105.389 73.309)
-		(width 0.2)
-		(layer "B.Cu")
-		(net 1)
-	)
-	(segment
 		(start 86.23 101)
 		(end 85.4553 101.7747)
@@
 	)
 	(segment
-		(start 113.009 75.849)
-		(end 114.16 77)
-		(width 0.2)
-		(layer "B.Cu")
-		(net 1)
-	)
-	(segment
 		(start 93.6 100.83)
 		(end 93.77 101)
@@
 	)
 	(segment
-		(start 88.76 74.46)
-		(end 89.916 75.616)
-		(width 0.2)
-		(layer "B.Cu")
-		(net 1)
-	)
-	(segment
 		(start 99.111 113.589)
 		(end 100.508 114.986)
@@
 	)
 	(segment
-		(start 96.38 77)
-		(end 97.531 75.849)
-		(width 0.2)
-		(layer "B.Cu")
-		(net 1)
-	)
-	(segment
 		(start 94.21 100.56)
 		(end 94.4431 100.3269)
@@
 	)
 	(segment
-		(start 105.389 73.309)
-		(end 106.54 74.46)
-		(width 0.2)
-		(layer "B.Cu")
-		(net 1)
-	)
-	(segment
-		(start 107.929 75.849)
-		(end 113.009 75.849)
-		(width 0.2)
-		(layer "B.Cu")
-		(net 1)
-	)
-	(segment
 		(start 94.4431 100.3269)
 		(end 96 100.3269)
@@
 		(net 71)
 	)
+	(zone
+		(net 1)
+		(net_name "GND")
+		(layer "B.Cu")
+		(hatch edge 0.5)
+		(connect_pads
+			(clearance 0)
+		)
+		(min_thickness 0.25)
+		(filled_areas_thickness no)
+		(fill yes
+			(mode hatch)
+			(thermal_gap 0.5)
+			(thermal_bridge_width 0.5)
+			(hatch_thickness 1)
+			(hatch_gap 1.5)
+			(hatch_orientation 0)
+			(hatch_border_algorithm hatch_thickness)
+			(hatch_min_hole_area 0.3)
+		)
+		(polygon
+			(pts
+				(xy 50.47 50.47) (xy 129.337 50.47) (xy 129.21 129.21) (xy 50.47 129.21)
+			)
+		)
+	)
 	(group ""
