File: kiCad/hat/dreamV1_0.kicad_pcb (KiCad board)
At the start: 2 copper layers, 80 x 80 mm, 37 parts, among them IC1 TGS2611-C00, J1 GPIO, J11 10132328-10011LF, J2 Qwiic_Vertical, J3 679305124022, J4 Qwiic_Vertical, J5 M20-7830542, J6 Qwiic_Vertical, J7 5013310607, J8 Qwiic_Vertical, J9 Qwiic_Vertical, Q1 BSS138, U1 AP2112K-3.3, U2 BME280, U3 INA219BxDCN

Commit message: update_hat
Parts:
- added B1: JST 2-PH, Capacitor_SMD:C_0201_0603Metric_Pad0.64x0.40mm_HandSolder, F.Cu at (194.1, 78.6)
- added C10: 2.2uF, Capacitor_SMD:C_0201_0603Metric_Pad0.64x0.40mm_HandSolder, F.Cu at (194.1, 83.9)
- added C11: 100uF, Capacitor_SMD:C_0201_0603Metric_Pad0.64x0.40mm_HandSolder, F.Cu at (194.1, 85.6)
- added C12: 10uF, Capacitor_SMD:C_0201_0603Metric_Pad0.64x0.40mm_HandSolder, F.Cu at (194.1, 87.4)
- added C8: 10uF, Capacitor_SMD:C_0201_0603Metric_Pad0.64x0.40mm_HandSolder, F.Cu at (194.1, 80.4)
- added C9: 0.1uF, Capacitor_SMD:C_0201_0603Metric_Pad0.64x0.40mm_HandSolder, F.Cu at (194.1, 82.1)
- added CHRG/LBO1: ORANGE, Capacitor_SMD:C_0201_0603Metric_Pad0.64x0.40mm_HandSolder, F.Cu at (194.1, 89.1)
- added DONE1: GREEN, Capacitor_SMD:C_0201_0603Metric_Pad0.64x0.40mm_HandSolder, F.Cu at (194.1, 90.9)
- added L1: 6.8uH, Inductor_SMD:L_0201_0603Metric, F.Cu at (186.6, 78.6)
- added LED1: RED, LED_SMD:LED_0201_0603Metric, F.Cu at (190.8, 91.6)
- added LED2: BLUE, LED_SMD:LED_0201_0603Metric, F.Cu at (190.8, 93.3)
- added R10: 1k, Resistor_SMD:R_0201_0603Metric, F.Cu at (186.6, 82.1)
- added R11: 1.87m, Resistor_SMD:R_0201_0603Metric, F.Cu at (186.6, 83.9)
- added R12: 340k, Resistor_SMD:R_0201_0603Metric, F.Cu at (186.6, 85.6)
- added R13: 200k, Resistor_SMD:R_0201_0603Metric, F.Cu at (189.0, 78.6)
- added R14: 270k, Resistor_SMD:R_0201_0603Metric, F.Cu at (189.0, 80.4)
- added R15: 100k, Resistor_SMD:R_0201_0603Metric, F.Cu at (189.0, 82.1)
- added R16: 1k, Resistor_SMD:R_0201_0603Metric, F.Cu at (189.0, 83.9)
- added R17: 100k, Resistor_SMD:R_0201_0603Metric, F.Cu at (189.0, 85.6)
- added R18: 1.87m, Resistor_SMD:R_0603_1608Metric, F.Cu at (187.3, 92.0)
- added R19: 200k, Resistor_SMD:R_0201_0603Metric, F.Cu at (191.5, 78.6)
- added R20: 1k, Resistor_SMD:R_0201_0603Metric, F.Cu at (191.5, 80.4)
- added R21: 1k, Resistor_SMD:R_0201_0603Metric, F.Cu at (191.5, 82.1)
- added R9: 1k, Resistor_SMD:R_0201_0603Metric, F.Cu at (186.6, 80.4)
- added T1: MMUN2133LT1G, Transistor_SmallSignal:SOT95P240X111-3N, F.Cu at (207.6, 96.4)
- added THERMO1: 15k, Resistor_SMD:R_0201_0603Metric, F.Cu at (191.5, 83.9)
- added U4: TPS61090RSAR, Package_DFN_QFN:Texas_S-PVQFN-N14, F.Cu at (211.3, 85.0)
- added U5: MCP73871, Package_DFN_QFN:QFN-20-1EP_3.5x3.5mm_P0.5mm_EP2x2mm, F.Cu at (209.3, 75.0)
- added X1: TERMBLOCK_1X2, Fuse:Fuse_1210_3225Metric, F.Cu at (188.1, 88.6)
- IC1: value TGS2611-C00 -> TGS2611; footprint KiCad:TGS2611C00 -> Sensor_Humidity:TO180P920H1340-4
- R1: renamed from R7; footprint downloaded:RC0603N_YAG-L -> Resistor_SMD:RESC1608X55N
- renumbered C2 to C1, C4 to C2, C5 to C3, C1 to C4, C3 to C5, C7 to C6, C6 to C7, J4 to J10, J11 to J2, J8 to J3, J2 to J4, J7 to J5, J3 to J6, J6 to J7, J5 to J8, JP2 to JP1, JP1 to JP2, R4 to R2, R5 to R3, R6 to R4, R8 to R5, R2 to R6, R1 to R7, R3 to R8, U3 to U1, U1 to U3
Routing:
- net Net-(U1-IN-): track 37.2 -> 0.00 mm
- net (no net): track 0.00 -> 37.2 mm
