File: kiCad/hat/dreamV1_0.kicad_pcb (KiCad board)
At the start: 2 copper layers, 54 parts, among them J1 GPIO, J2 10132328-10011LF, Q1 BSS138, T1 MMUN2133LT1G, U1 INA219BxDCN, U2 BME280, U3 AP2112K-3.3, U4 TPS61090RSAR, U5 MCP73871, X1 TERMBLOCK_1X2

Commit message: update hat
Parts:
- removed the C8 at (140.6, 63.2)
- removed the C9 at (132.4, 63.5)
- removed T1: MMUN2133LT1G, Transistor_SmallSignal:SOT95P240X111-3N
- removed X1: TERMBLOCK_1X2, Fuse:Fuse_1210_3225Metric
- added Q2: MMUN2133LT1G, MMUN2133LT1G:SOT95P240X111-3N, B.Cu at (127.9, 63.2)
- C10, C11, R13, R14, R15: moved to B.Cu
- R18, R19: footprint Resistor_SMD:R_0603_1608Metric -> Resistor_SMD:R_0201_0603Metric_Pad0.64x0.40mm_HandSolder; moved to B.Cu
- moved R20 152.5 mm to (119.4, 59.4), turned to -90 degrees
- moved R13 140.6 mm to (117.7, 65.5), turned to 180 degrees
- moved LED1 117.7 mm to (117.8, 56.8), turned to 180 degrees
- moved C10 112.9 mm to (127.2, 66.9), turned to -90 degrees
- moved C11 112.1 mm to (128.2, 66.9), turned to -90 degrees
- moved R15 22.6 mm to (106.3, 69.5), turned to 180 degrees
- moved R14 21.5 mm to (106.3, 72.1), turned to 180 degrees
- moved R19 7.92 mm to (121.4, 63.0), turned to -90 degrees
- moved R4 4.58 mm to (117.7, 59.4), turned to -90 degrees
- moved R1 4.56 mm to (115.9, 59.4), turned to -90 degrees
- moved R18 2.68 mm to (122.1, 63.0), turned to 90 degrees
- moved U5 2.26 mm to (112.6, 70.2)
Connections:
- net /ENABLE renamed Net-(U4-EN)
- net SW renamed Net-(L1-2)
- L1 pad 2: (no net) -> VBAT
- LED1 pad : (no net) -> GND
- LED1 pad 1: (no net) -> Net-(LED1-PadA)
- U5 pad CE: (no net) -> 5V_BUS_USB
- U5 pad VIN1: (no net) -> 5V_BUS_USB
- U5 pad VIN2: (no net) -> 5V_BUS_USB
Routing:
- net GND: track 46.9 -> 69.0 mm, vias 5 -> 6
- net VBAT: track 25.4 -> 39.9 mm, vias 0 -> 3
- net /LBO: track 0.00 -> 11.4 mm
- net Net-(Q2-C): track 0.00 -> 11.4 mm, vias 0 -> 1
- net 5.0V: track 2.25 -> 13.3 mm
- net 5V_BUS_USB: track 19.8 -> 26.6 mm
- net Net-(J2-CC1): track 14.4 -> 11.0 mm
- net (no net): track 0.00 -> 3.29 mm
- net Net-(LED1-PadA): track 0.00 -> 2.26 mm
- net Net-(U4-FB): track 0.00 -> 2.14 mm
- net Net-(U4-EN): track 0.00 -> 2.07 mm
- net Net-(J2-CC2): track 16.3 -> 15.6 mm

Commit message: added some to scale drawings for layout design
Parts:
- added C8: 10uF, Capacitor_SMD:C_0201_0603Metric_Pad0.64x0.40mm_HandSolder, F.Cu at (200.5, 65.4)
- added C9: 0.1uF, Capacitor_SMD:C_0201_0603Metric, F.Cu at (234.2, 51.0)
- added G***: LOGO, LOGO, F.Cu at (118.2, 100.2)
- added G***: LOGO, LOGO, F.Cu at (140.5, 99.7)
- added G***: LOGO, LOGO, B.Cu at (-71.5, 179.7)
- added G***: LOGO, LOGO, B.Cu at (-75.4, 138.0)
- added J1: GPIO, Connector_PinSocket_2.54mm:PinSocket_2x20_P2.54mm_Vertical, F.Cu at (-47.0, 162.0)
- moved J1 136.1 mm to (-50.9, 120.4), turned to -90 degrees
- moved R10 82.8 mm to (202.9, 51.6)
- moved R16 82.8 mm to (203.2, 59.2)
- moved R21 82.8 mm to (210.8, 52.9)
- moved R9 82.8 mm to (201.9, 47.8)
- moved THERMO1 82.8 mm to (212.1, 58.0)
- moved C1 53.3 mm to (227.4, 123.0)
- moved C2 50.3 mm to (226.8, 122.2)
- moved C3 44.1 mm to (206.1, 90.5)
- moved AP2112K-3.3 43.5 mm to (207.7, 114.7)
- moved INA219 41.1 mm to (215.0, 112.1)
- moved Q1 41.0 mm to (224.3, 114.3)
- moved R3 41.0 mm to (205.9, 107.3)
- moved RGBLED 41.0 mm to (216.6, 123.2)
- moved R7 41.0 mm to (207.7, 120.6)
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- renumbered U3 to AP2112K-3.3, U2 to BME280, U1 to INA219, D1 to RGBLED
Connections:
- L1 pad 1: Net-(L1-2) -> (no net)
- L1 pad 2: VBAT -> (no net)
- LED1 pad : GND -> (no net)
- LED1 pad 1: Net-(LED1-PadA) -> (no net)
- U4 pad LBI: Net-(U4-LBI) -> (no net)
- U5 pad CE: 5V_BUS_USB -> (no net)
- U5 pad VIN1: 5V_BUS_USB -> (no net)
- U5 pad VIN2: 5V_BUS_USB -> (no net)
Routing:
- net GND: track 69.0 -> 0.00 mm, vias 6 -> 0
- net VBAT: track 39.9 -> 0.00 mm, vias 3 -> 0
- net 5V_BUS_USB: track 26.6 -> 0.00 mm, vias 4 -> 0
- net Net-(J2-CC2): track 15.6 -> 0.21 mm
- net 5.0V: track 13.3 -> 0.00 mm
- net /LBO: track 11.4 -> 0.00 mm
- net Net-(Q2-C): track 11.4 -> 0.00 mm, vias 1 -> 0
- net Net-(J2-CC1): track 11.0 -> 0.00 mm
- net (no net): track 3.29 -> 0.00 mm
- net Net-(LED1-PadA): track 2.26 -> 0.00 mm
- net Net-(U4-FB): track 2.14 -> 0.00 mm
- net Net-(U4-LBI): track 2.11 -> 0.00 mm
- net Net-(U4-EN): track 2.07 -> 0.00 mm
- net Net-(L1-2): track 1.96 -> 0.00 mm
Other:
- board outline added: 80 x 80 mm
- copper layers 2 -> 4
