File: kiCad/hat/_autosave-dreamV1_0.kicad_pcb (KiCad board)
At the start: 2 copper layers, 54 parts, among them J1 GPIO, J2 10132328-10011LF, Q1 BSS138, T1 MMUN2133LT1G, U1 INA219BxDCN, U2 BME280, U3 AP2112K-3.3, U4 TPS61090RSAR, U5 MCP73871, X1 TERMBLOCK_1X2

Commit message: update hat; PCB reset
Parts:
- removed T1: MMUN2133LT1G, Transistor_SmallSignal:SOT95P240X111-3N
- removed X1: TERMBLOCK_1X2, Fuse:Fuse_1210_3225Metric
- added Q2: MMUN2133LT1G, MMUN2133LT1G:SOT95P240X111-3N, F.Cu at (127.0, 63.3)
- R18, R19: footprint Resistor_SMD:R_0603_1608Metric -> Resistor_SMD:R_0201_0603Metric_Pad0.64x0.40mm_HandSolder; moved to B.Cu
- moved R19 7.92 mm to (121.4, 63.0), turned to -90 degrees
- moved R1 5.24 mm to (115.2, 59.4), turned to -90 degrees
- moved R4 5.04 mm to (117.0, 59.4), turned to -90 degrees
- moved R18 2.68 mm to (122.1, 63.0), turned to 90 degrees
Connections:
- L1 pad 1: SW -> (no net)
- U4 pad 3: SW -> Net-(L1-2)
- U4 pad 4: SW -> Net-(L1-2)
Routing:
- net Net-(J2-CC1): track 14.4 -> 3.61 mm
- net Net-(J2-CC2): track 16.3 -> 6.45 mm
- net GND: track 46.9 -> 50.2 mm
- net 5.0V: track 2.25 -> 5.37 mm
- net Net-(U4-FB): track 0.00 -> 2.14 mm
- net SW: track 1.96 -> 0.00 mm
- net Net-(L1-2): track 0.00 -> 1.96 mm
