File: kiCad/hat/dreamV1_0.kicad_sch (KiCad schematic)
At the start: 35 parts, among them IC1 TGS2611-C00, J1 GPIO, J11 10132328-10011LF, J2 Qwiic_Vertical, J3 679305124022, J4 Qwiic_Vertical, J5 M20-7830542, J6 Qwiic_Vertical, J7 5013310607, J8 Qwiic_Vertical, J9 Qwiic_Vertical, Q1 BSS138, U1 AP2112K-3.3, U2 BME280, U3 INA219BxDCN

Commit message: update_hat
Parts:
- added B1: JST 2-PH, Capacitor_SMD:C_0201_0603Metric_Pad0.64x0.40mm_HandSolder, symbol Adafruit PowerBoost 1000C Rev B-eagle-import:BATTERY
- added C10: 2.2uF, Capacitor_SMD:C_0201_0603Metric_Pad0.64x0.40mm_HandSolder, symbol Adafruit PowerBoost 1000C Rev B-eagle-import:CAP_CERAMIC0805-NOOUTLINE
- added C11: 100uF, Capacitor_SMD:C_0201_0603Metric_Pad0.64x0.40mm_HandSolder, symbol Adafruit PowerBoost 1000C Rev B-eagle-import:C-USC1210
- added C12, C8: 10uF, Capacitor_SMD:C_0201_0603Metric_Pad0.64x0.40mm_HandSolder, symbol Adafruit PowerBoost 1000C Rev B-eagle-import:CAP_CERAMIC0805-NOOUTLINE
- added C9: 0.1uF, Capacitor_SMD:C_0201_0603Metric_Pad0.64x0.40mm_HandSolder, symbol Adafruit PowerBoost 1000C Rev B-eagle-import:CAP_CERAMIC0805_10MGAP
- added CHRG/LBO1: ORANGE, Capacitor_SMD:C_0201_0603Metric_Pad0.64x0.40mm_HandSolder, symbol Adafruit PowerBoost 1000C Rev B-eagle-import:LED0805_NOOUTLINE
- added DONE1: GREEN, Capacitor_SMD:C_0201_0603Metric_Pad0.64x0.40mm_HandSolder, symbol Adafruit PowerBoost 1000C Rev B-eagle-import:LED0805_NOOUTLINE
- added L1: 6.8uH, Inductor_SMD:L_0201_0603Metric, symbol Adafruit PowerBoost 1000C Rev B-eagle-import:INDUCTORTDK_VLC5045
- added LED1: RED, LED_SMD:LED_0201_0603Metric, symbol Adafruit PowerBoost 1000C Rev B-eagle-import:LED0805_NOOUTLINE
- added LED2: BLUE, LED_SMD:LED_0201_0603Metric, symbol Adafruit PowerBoost 1000C Rev B-eagle-import:LED0805_NOOUTLINE
- added R10, R16, R20, R21, R9: 1k, Resistor_SMD:R_0201_0603Metric, symbol SparkFun-Resistor:10k_0603
- added R11: 1.87m, Resistor_SMD:R_0201_0603Metric, symbol SparkFun-Resistor:10k_0603
- added R12: 340k, Resistor_SMD:R_0201_0603Metric, symbol SparkFun-Resistor:10k_0603
- added R13, R19: 200k, Resistor_SMD:R_0201_0603Metric, symbol SparkFun-Resistor:10k_0603
- added R14: 270k, Resistor_SMD:R_0201_0603Metric, symbol SparkFun-Resistor:10k_0603
- added R15, R17: 100k, Resistor_SMD:R_0201_0603Metric, symbol SparkFun-Resistor:10k_0603
- added R18: 1.87m, Resistor_SMD:R_0603_1608Metric, symbol SparkFun-Resistor:10k_0603
- added T1: MMUN2133LT1G, Transistor_SmallSignal:SOT95P240X111-3N, symbol Adafruit PowerBoost 1000C Rev B-eagle-import:-PNP_DRIVER-SC59-BEC
- added THERMO1: 15k, Resistor_SMD:R_0201_0603Metric, symbol SparkFun-Resistor:10k_0603
- added U4: TPS61090RSAR, Package_DFN_QFN:Texas_S-PVQFN-N14, symbol Adafruit PowerBoost 1000C Rev B-eagle-import:VREG_TPS6103X
- added U5: MCP73871, Package_DFN_QFN:QFN-20-1EP_3.5x3.5mm_P0.5mm_EP2x2mm, symbol Adafruit PowerBoost 1000C Rev B-eagle-import:MCP73871
- added X1: TERMBLOCK_1X2, Fuse:Fuse_1210_3225Metric, symbol Adafruit PowerBoost 1000C Rev B-eagle-import:TERMBLOCK_1X2
- IC1: footprint TGS2611C00 -> Sensor_Humidity:TO180P920H1340-4
- R1: renamed from R7; footprint RC0603N_YAG-L -> Resistor_SMD:RESC1608X55N
- renumbered C2 to C1, C4 to C2, C5 to C3, C1 to C4, C3 to C5, C7 to C6, C6 to C7, J4 to J10, J11 to J2, J8 to J3, J2 to J4, J7 to J5, J3 to J6, J6 to J7, J5 to J8, JP2 to JP1, JP1 to JP2, R4 to R2, R5 to R3, R6 to R4, R8 to R5, R2 to R6, R1 to R7, R3 to R8, U3 to U1, U1 to U3
Connections:
- net GND: now also B1.1 (-), C10.2, C11.2, C12.2, C8.2, C9.2, LED1.C, LED2.C, R12.1, R15.1, R16.1, R17.1, R19.1, THERMO1.1, U4.10 (SYNC), U4.13 (GND), U4.5 (PGND), U4.6 (PGND), U4.7 (PGND), U4.P$18 (PGND), U4.P$19 (PGND), U4.P$20 (PGND), U4.P$21 (PGND), U4.P$22 (PGND), U4.THERMAL (PGND), U5.P$10 (VSS1), U5.P$11 (VSS2), U5.P$21 (THERMAL), X1.1
- new net: R14.1, R15.2, U5.P$2 (VPCC)
- new net: DONE1.C, R10.2
- new net: R17.2, U5.P$12 (PROG3)
- new net: R16.2, U5.P$13 (PROG1)
- new net: THERMO1.2, U5.P$5 (THERM)
- new net: R10.1, U5.P$7 (STAT2)
- new net: R9.1, U5.P$8 (STAT1/LBO)
- new net: LED2.A, R21.1
- new net: CHRG/LBO1.C, R9.2
- new net: R11.1, R12.2, U4.9 (LBI)
- new net: LED1.A, R20.1
- new net: R20.2, T1.C
- new net: L1.P$2 (2), U4.3 (SW), U4.4 (SW)
- new net: R18.1, R19.2, U4.14 (FB)
- new net 5.0V: C10.1, C11.1, R18.2, R21.2, U4.1 (VOUT), U4.15 (VOUT), U4.16 (VOUT), X1.2
- new net ENABLE: R13.1, U4.11 (EN)
- new net LBO: T1.B, U4.12 (LBO)
- new net VBAT: C8.1, C9.1, L1.P$1 (1), R11.2, R13.2, T1.E, U4.8 (VBAT), U5.P$1 (VOUT1), U5.P$20 (VOUT2)
- new net VBUS: CHRG/LBO1.A, DONE1.A, R14.2, U5.P$17 (CE), U5.P$18 (VIN1), U5.P$19 (VIN2), U5.P$3 (SEL), U5.P$4 (PROG2), U5.P$9 (/TE)
- new net VLIPO: B1.2 (+), C12.1, U5.P$14 (VBAT1), U5.P$15 (VBAT2), U5.P$16 (VBATSENS)
Other:
- note added: "1.0K = 1000mA"
- note added: "10K NTC Thermistor:"
- note added: "2.0K = 500mA"
- note added: "6.8uH power w/2A current"
- note added: "Boost Converter"
- note added: "Both grounds must be connected on the PCB at only one point close to the GND pin."
- note added: "Charge Rate = 1000V/PROG1"
- note added: "No Thermistor:"
- note added: "On/Off Switch"
- note added: "R3 = 1.9Mohm for 5.2V R3 = 1.1Mohm for 3.3V"
- note added: "RT1 = 0, RT2 = 10K"
- note added: "RT1 = TBD, RT2 = TBD"
- note added: "See Pg 15 1st para"
- note added: "USB/AC Battery Charger w/ Power Path Management"

Commit message: update hat; PCB reset
Parts:
- removed T1: MMUN2133LT1G, Transistor_SmallSignal:SOT95P240X111-3N, symbol Adafruit PowerBoost 1000C Rev B-eagle-import:-PNP_DRIVER-SC59-BEC
- removed X1: TERMBLOCK_1X2, Fuse:Fuse_1210_3225Metric, symbol Adafruit PowerBoost 1000C Rev B-eagle-import:TERMBLOCK_1X2
- added C13: 10uF, SparkFun-Capacitor:C_0603_1608Metric, symbol SparkFun-Capacitor:C
- added Q2: MMUN2133LT1G, MMUN2133LT1G:SOT95P240X111-3N, symbol MMUN2133LT1G:MMUN2133LT1G
- C10, C11, C9: footprint Capacitor_SMD:C_0201_0603Metric_Pad0.64x0.40mm_HandSolder -> Capacitor_SMD:C_0201_0603Metric
- J2: footprint downloaded:10132328-10011LF -> Connector_USB:USB_C_Receptacle_Molex_105450-0101
- R10, R13, R14, R15, R16, R17, R20, R21, R9, THERMO1: footprint Resistor_SMD:R_0201_0603Metric -> Resistor_SMD:R_0603_1608Metric
- R11, R12, R19: footprint Resistor_SMD:R_0201_0603Metric -> Resistor_SMD:R_0201_0603Metric_Pad0.64x0.40mm_HandSolder
- R18: footprint Resistor_SMD:R_0603_1608Metric -> Resistor_SMD:R_0201_0603Metric_Pad0.64x0.40mm_HandSolder
- R4: footprint downloaded:RC0603N_YAG-L -> Resistor_SMD:RESC1608X55N
- U4: footprint Package_DFN_QFN:Texas_S-PVQFN-N14 -> TPS61090RSAR:QFN65P400X400X100-17N; Vendor (none) -> https://www.digikey.com/en/products/detail/texas-instrument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
Connections:
- net 5V_BUS_USB: now also CHRG/LBO1.A, DONE1.A, R14.2, U5.P$17 (CE), U5.P$3 (SEL), U5.P$4 (PROG2), U5.P$9 (/TE), C13.2
- net GND: now also C13.1
- net LBO: now also Q2.1 (B)
- net VBAT: now also Q2.2 (E)
- net VBUS: no longer CHRG/LBO1.A, DONE1.A, R14.2, U5.P$17 (CE), U5.P$3 (SEL), U5.P$4 (PROG2), U5.P$9 (/TE)
- net at R20.2: now also Q2.3 (C)
- net ENABLE: no longer names the net of R13.1, U4.11 (EN)
Other:
- moved on the sheet: R13

Commit message: update hat
Parts:
- removed LED2: BLUE, LED_SMD:LED_0201_0603Metric, symbol Adafruit PowerBoost 1000C Rev B-eagle-import:LED0805_NOOUTLINE
- removed R21: 1k, Resistor_SMD:R_0603_1608Metric, symbol SparkFun-Resistor:10k_0603
Connections:
- net VBUS is gone; now on net 5V_BUS_USB: U5.P$18 (VIN1), U5.P$19 (VIN2)
