File: kiCad/dreamV2_0/dreamV1_0.kicad_pcb (KiCad board)
At the start: 2 copper layers, 79 x 78.9 mm, 36 parts, among them IC1 TGS2611-C00, J1 GPIO, J11 10132328-10011LF, J2 Qwiic_Vertical, J3 679305124022, J4 Qwiic_Vertical, J5 M20-7830542, J6 Qwiic_Vertical, J7 5013310607, J8 Qwiic_Vertical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

Commit message: Updated gerber
Routing:
- net +3V3: track 167.7 -> 174.3 mm
Changed lines of the file:
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@@
 		(grid_origin 100 100)
 		(pcbplotparams
-			(layerselection 0x00000000_00000000_55555555_5755f5ff)
+			(layerselection 0x00000000_00000000_55555555_5757f5ff)
 			(plot_on_all_layers_selection 0x00000000_00000000_00000000_00000000)
 			(disableapertmacros no)
@@
 			(at 3.75 0 180)
 			(size 0.58 0.58)
-			(drill 0.58)
+			(drill 0.66)
 			(layers "*.Mask")
 		)
@@
 		)
 	)
-	(gr_line
-		(start 62.535 86.157)
-		(end 62.535 93.777)
-		(stroke
-			(width 0.3)
-			(type solid)
-		)
-		(layer "F.Cu")
-		(net 31)
-	)
 	(gr_rect
 		(start 100 79)
@@
 	)
 	(segment
+		(start 62.54 89.54)
+		(end 64.656 91.656)
+		(width 0.2)
+		(layer "F.Cu")
+		(net 31)
+	)
+	(segment
 		(start 60.5665 121.6535)
 		(end 59.995 121.6535)
@@
 	)
 	(segment
-		(start 58.09 98.222)
+		(start 64.656 91.656)
 		(end 67.615 88.697)
 		(width 0.3)
@@
 	)
 	(segment
+		(start 62.54 86.02)
+		(end 62.54 89.54)
+		(width 0.2)
+		(layer "F.Cu")
+		(net 31)
+	)
+	(segment
 		(start 58.09 111.8225)
 		(end 58.09 98.222)
@@
 	)
 	(segment
+		(start 58.09 98.222)
+		(end 64.656 91.656)
+		(width 0.3)
+		(layer "F.Cu")
+		(net 31)
+	)
+	(segment
 		(start 64.476 125.563)
 		(end 60.5665 121.6535)
@@
 		(start 93.5 57.089004)
 		(end 107.096996 57.089004)
-		(width 0.8)
+		(width 0.7)
 		(layer "F.Cu")
 		(net 55)
@@
 		(start 92.830998 56.420002)
 		(end 93.5 57.089004)
-		(width 0.4)
+		(width 0.3)
 		(layer "F.Cu")
 		(net 55)
@@
 		(members "82ff541d-485a-4c8c-afc1-b71808d85e91" "9312597b-e66a-423b-b6f1-8e8861bbc515")
 	)
+	(group ""
+		(members "fede43f0-8fa0-4d7c-bbdf-32c1e14aa9e4")
+	)
 	(embedded_fonts no)
