File: kiCad/dreamV3_0/Dream_V3_0/Dream_V3_0.kicad_sch (KiCad schematic)
At the start: 43 parts, among them IC1 TGS2611-C00, J1 GPIO, J11 10132328-10011LF, J2 Qwiic_Vertical, J3 679305124022, J4 Qwiic_Vertical, J5 M20-7830542, J6 Qwiic_Vertical, J7 5013310607, J8 Qwiic_4pin_Vertical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

Commit message: update structure
Connections:
- net GPIO23/SDA4: now also Q2.3 (D), R13.3
- net GPIO24/SCL4: now also Q2.6 (D), R13.1
- net GPIO5/SDA5: no longer Q2.3 (D), R13.3
- net GPIO6/SCL5: no longer Q2.6 (D), R13.1
Changed lines of the file:
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@@
 		)
 	)
-	(label "GPIO6{slash}SCL5"
+	(label "GPIO24{slash}SCL4"
 		(at 101.6 81.28 0)
 		(effects
@@
 		)
 	)
-	(label "GPIO5{slash}SDA5"
+	(label "GPIO23{slash}SDA4"
 		(at 101.6 67.31 0)
 		(effects
