File: kiCad/dreamV3_0/Dream_leov1.kicad_pcb (KiCad board)
At the start: 2 copper layers, 80 x 80 mm, 38 parts, among them IC1 TGS2611-C00, J1 GPIO, J11 10132328-10011LF, J2 Qwiic_Vertical, J3 679305124022, J4 Qwiic_Vertical, J5 M20-7830542, J6 Qwiic_Vertical, J7 5013310607, Q1 BSS138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

Commit message: final john update
Parts:
- added G***: LOGO, LOGO, F.Cu at (64.0, 23.5)
- C3: moved to F.Cu
- moved C3 38.0 mm to (100.0, 91.0)
- moved U1 15.7 mm to (93.5, 79.5)
- moved R11 8.69 mm to (102.5, 76.0), turned to -90 degrees
- moved R4 7.13 mm to (94.5, 75.5), turned to 90 degrees
- moved U4 6.52 mm to (100.0, 93.5)
- moved C1 6.50 mm to (82.5, 91.0)
- moved R5 5.54 mm to (78.5, 82.0), turned to 180 degrees
- moved U2 5.48 mm to (82.5, 93.5)
- moved JP1 4.61 mm to (79.0, 93.0)
- moved C7 0.68 mm to (99.8, 69.4)
- moved C5 0.50 mm to (82.5, 82.0), turned to 90 degrees
- renumbered j9 to J9
Connections:
- C2 pad 1: +3.3V -> +3V3
- J1 pad : (no net) -> +3.3V
- J1 pad 17: +3.3V -> +3V3
- J2 pad 2: +3.3V -> +3V3
- J2 pad 3: /GPIO5/SDA5 -> /GPIO2/SDA1
- J4 pad 3: /GPIO27/SDA3 -> /GPIO5/SDA5
- J4 pad 4: /GPIO22/SCL3 -> /GPIO6/SCL5
- J6 pad 2: +3.3V -> +3V3
- J9 pad 2: +3.3V -> +3V3
- J9 pad 3: /GPIO2/SDA1 -> /GPIO27/SDA3
- J9 pad 4: /GPIO3/SCL1 -> /GPIO22/SCL3
- JP1 pad 2: /BME_ADD -> /BME_ADD_1
- Q1 pad 1: /BME_SCL -> /BME_SCL1
- Q1 pad 4: /BME_SDA -> /BME_SDA1
- R1 pad 2: +3.3V -> +3V3
- R1 pad 4: +3.3V -> +3V3
- R1 pad 5: /BME_SCL -> /BME_SCL1
- R1 pad 8: /BME_SDA -> /BME_SDA1
- U1 pad 1: +3.3V -> +3V3
- U1 pad en: (no net) -> +3V3
- U2 pad 3: /BME_SDA -> /BME_SDA2
- U2 pad 4: /BME_SCL -> /BME_SCL2
- U2 pad 5: /BME_ADD -> /BME_ADD_2
- U4 pad 6: +3.3V -> BME_3V3
- U4 pad 8: +3.3V -> BME_3V3
Routing:
- net +3.3V: track 188.0 -> 6.62 mm, vias 8 -> 0
- net +5V: track 258.0 -> 159.6 mm, vias 5 -> 1
- net GND: track 261.5 -> 166.1 mm, vias 6 -> 4
- net +3V3: track 0.00 -> 70.9 mm, vias 0 -> 3
- net /GPIO27/SDA3: track 99.2 -> 60.6 mm
- net /GPIO22/SCL3: track 98.2 -> 59.6 mm
- net /GPIO23/SDA4: track 30.5 -> 66.9 mm, vias 1 -> 2
- net /GPIO24/SCL4: track 33.5 -> 69.6 mm, vias 1 -> 2
- net /BME_SCL: track 33.1 -> 0.00 mm, vias 2 -> 0
- net /GPIO6/SCL5: track 74.0 -> 47.1 mm, vias 4 -> 3
- net /BME_SDA: track 24.5 -> 0.00 mm, vias 2 -> 0
- net /GPIO5/SDA5: track 75.7 -> 53.7 mm, vias 4 -> 3
- net BME_3V3: track 6.27 -> 27.1 mm
- net /INA+: track 12.9 -> 0.00 mm, vias 1 -> 0
- net /INA_ADD0: track 9.77 -> 0.00 mm
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Other:
- outline, holes or cut-outs redrawn
- board text added: "- - -"
- board text added: "DREAM V3"
- board text added: "Lakitha Wijeratne John Phelan Leonardo Murillo"
- board text added: "MINTS-AI DREAM V3"
- board text removed: "- - - - -"
