File: kiCad/dreamV3_0/Dream_V3.kicad_pcb (KiCad board)
At the start: 2 copper layers, 80 x 80 mm, 44 parts, among them IC1 TGS2611-C00, J1 GPIO, J11 10132328-10011LF, J2 Qwiic_Vertical, J3 679305124022, J4 Qwiic_Vertical, J5 M20-7830542, J6 Qwiic_Vertical, J7 5013310607, J8 Qwiic_4pin_Vertical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

Commit message: Final DreamV3
Routing:
- net GND: track 218.3 -> 207.3 mm
Other:
- outline, holes or cut-outs redrawn
- board text added: "PWR"
- board text added: "U"

Commit message: Final DreamV3
Parts:
- S1: value NK236 -> OS102011MA1QN1
Other:
- board text added: "OFF"
- board text added: "ON"
Changed lines of the file:
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@@
 			)
 		)
-		(property "Value" "NK236"
+		(property "Value" "OS102011MA1QN1"
 			(at 1.7 7.7 0)
 			(layer "F.Fab")
@@
 			)
 		)
-		(property "Datasheet" "NK236"
+		(property "Datasheet" "https://www.littelfuse.com/assetdocs/littelfuse-c-k-slide-os-series-datasheet?assetguid=f8954ac2-65ba-431f-af55-b0493370575e"
 			(at 0 0 180)
 			(unlocked yes)
@@
 			)
 		)
-		(property "Description" "Pushbutton Switches OFF-(ON) .201 RD CAP RIGHT ANGL PC .4VA Process Sealed Subminiature Pushbuttons"
+		(property "Description" "Slide Switch SPDT Through Hole, Right Angle"
 			(at 0 0 180)
 			(unlocked yes)
@@
 			)
 		)
-		(property "SnapEDA_Link" "https://www.snapeda.com/parts/500ASSP1M6QE/E-Switch/view-part/?ref=snap"
-			(at 0 0 180)
-			(unlocked yes)
-			(layer "F.Fab")
-			(hide yes)
-			(effects
-				(font
-					(size 1 1)
-					(thickness 0.15)
-				)
-			)
-		)
-		(property "MP" "500ASSP1M6QE"
-			(at 0 0 180)
-			(unlocked yes)
-			(layer "F.Fab")
-			(hide yes)
-			(effects
-				(font
-					(size 1 1)
-					(thickness 0.15)
-				)
-			)
-		)
-		(property "Description_1" "Slide Switch, 500A Series, SPDT, ON-ON, 3A, 120VAC/28VDC, Silver, R/A, PC Pin | E-Switch 500ASSP1M6QE"
-			(at 0 0 180)
-			(unlocked yes)
-			(layer "F.Fab")
-			(hide yes)
-			(effects
-				(font
-					(size 1 1)
-					(thickness 0.15)
-				)
-			)
-		)
-		(property "MANUFACTURER" "E-Switch"
-			(at 0 0 180)
-			(unlocked yes)
-			(layer "F.Fab")
-			(hide yes)
-			(effects
-				(font
-					(size 1 1)
-					(thickness 0.15)
-				)
-			)
-		)
-		(property "Availability" "In Stock"
-			(at 0 0 180)
-			(unlocked yes)
-			(layer "F.Fab")
-			(hide yes)
-			(effects
-				(font
-					(size 1 1)
-					(thickness 0.15)
-				)
-			)
-		)
-		(property "SNAPEDA_PN" "500ASSP1M6QE"
-			(at 0 0 180)
-			(unlocked yes)
-			(layer "F.Fab")
-			(hide yes)
-			(effects
-				(font
-					(size 1 1)
-					(thickness 0.15)
-				)
-			)
-		)
-		(property "Height" "6.18"
-			(at 0 0 180)
-			(unlocked yes)
-			(layer "F.Fab")
-			(hide yes)
-			(effects
-				(font
-					(size 1 1)
-					(thickness 0.15)
-				)
-			)
-		)
-		(property "Mouser Part Number" "633-AB11AH-FC"
-			(at 0 0 180)
-			(unlocked yes)
-			(layer "F.Fab")
-			(hide yes)
-			(effects
-				(font
-					(size 1 1)
-					(thickness 0.15)
-				)
-			)
-		)
-		(property "Mouser Price/Stock" "https://www.mouser.co.uk/ProductDetail/NKK-Switches/AB11AH-FC?qs=E3XkhTW0K2FjNZbXLHs%252BZw%3D%3D"
-			(at 0 0 180)
-			(unlocked yes)
-			(layer "F.Fab")
-			(hide yes)
-			(effects
-				(font
-					(size 1 1)
-					(thickness 0.15)
-				)
-			)
-		)
-		(property "Manufacturer_Name" "NKK Switches"
-			(at 0 0 180)
-			(unlocked yes)
-			(layer "F.Fab")
-			(hide yes)
-			(effects
-				(font
-					(size 1 1)
-					(thickness 0.15)
-				)
-			)
-		)
-		(property "Manufacturer_Part_Number" "AB11AH-FC"
-			(at 0 0 180)
-			(unlocked yes)
-			(layer "F.Fab")
-			(hide yes)
-			(effects
-				(font
-					(size 1 1)
-					(thickness 0.15)
-				)
-			)
-		)
-		(property "Vendor" "https://www.digikey.com/en/products/detail/nkk-switches/AB11AH-FC/1055910?s=N4IgTCBcDaIIICECMS4AkC0AxAwiAugL5A"
-			(at 0 0 180)
-			(unlocked yes)
-			(layer "F.Fab")
-			(hide yes)
-			(effects
-				(font
-					(size 1 1)
-					(thickness 0.15)
-				)
-			)
-		)
-		(property "MF" "E-Switch"
-			(at 0 0 180)
-			(unlocked yes)
-			(layer "F.Fab")
-			(hide yes)
-			(effects
-				(font
-					(size 1 1)
-					(thickness 0.15)
-				)
-			)
-		)
-		(property "MAXIMUM_PACKAGE_HEIGHT" "5.59 mm"
-			(at 0 0 180)
-			(unlocked yes)
-			(layer "F.Fab")
-			(hide yes)
-			(effects
-				(font
-					(size 1 1)
-					(thickness 0.15)
-				)
-			)
-		)
-		(property "Package" "None"
-			(at 0 0 180)
-			(unlocked yes)
-			(layer "F.Fab")
-			(hide yes)
-			(effects
-				(font
-					(size 1 1)
-					(thickness 0.15)
-				)
-			)
-		)
-		(property "Price" "None"
-			(at 0 0 180)
-			(unlocked yes)
-			(layer "F.Fab")
-			(hide yes)
-			(effects
-				(font
-					(size 1 1)
-					(thickness 0.15)
-				)
-			)
-		)
-		(property "Check_prices" "https://www.snapeda.com/parts/500ASSP1M6QE/E-Switch/view-part/?ref=eda"
-			(at 0 0 180)
+		(property "Manufacturer" "C&K"
+			(at 0 0 0)
 			(unlocked yes)
 			(layer "F.Fab")
@@
 			)
 		)
-		(property "STANDARD" "Manufacturer Recommendations"
-			(at 0 0 180)
+		(property "Vendor" "https://www.digikey.com/en/products/detail/c-k/OS102011MA1QN1/1981430"
+			(at 0 0 0)
 			(unlocked yes)
 			(layer "F.Fab")
@@
 			)
 		)
-		(property "PARTREV" "C"
-			(at 0 0 180)
+		(property "Product Number" "OS102011MA1QN1"
+			(at 0 0 0)
 			(unlocked yes)
 			(layer "F.Fab")
@@
 		)
 	)
+	(gr_text "OFF"
+		(at 106.5 22.5 0)
+		(layer "F.SilkS")
+		(effects
+			(font
+				(size 1.5 1.5)
+				(thickness 0.3)
+				(bold yes)
+			)
+			(justify left bottom)
+		)
+	)
 	(gr_text "I2C 4"
 		(at 122.5 31 0)
@@
 		)
 	)
+	(gr_text "ON"
+		(at 123 22.5 0)
+		(layer "F.SilkS")
+		(effects
+			(font
+				(size 1.5 1.5)
+				(thickness 0.3)
+				(bold yes)
+			)
+			(justify left bottom)
+		)
+	)
 	(gr_text "IPS7100"
 		(at 106.5 99 90)
@@
 	)
 	(gr_text "- - -"
-		(at 94.5 41.5 90)
+		(at 94.5 42 90)
 		(layer "F.SilkS")
 		(effects

Commit message: Final DreamV3
Routing:
- net GND: track 207.3 -> 173.7 mm
Changed lines of the file:
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@@
 		(capping no)
 		(filling no)
+		(zone_defaults)
 		(pcbplotparams
 			(layerselection 0x00000000_00000000_55555555_5755f5ff)
@@
 		)
 	)
+	(dimension
+		(type orthogonal)
+		(layer "Dwgs.User")
+		(pts
+			(xy 55.5 96.5) (xy 129.5 96.5)
+		)
+		(height 8.5)
+		(orientation 0)
+		(format
+			(prefix "")
+			(suffix "")
+			(units 3)
+			(units_format 0)
+			(precision 4)
+			(suppress_zeroes yes)
+		)
+		(style
+			(thickness 0.1)
+			(arrow_length 1.27)
+			(text_position_mode 0)
+			(arrow_direction outward)
+			(extension_height 0.58642)
+			(extension_offset 0.5)
+			(keep_text_aligned yes)
+		)
+		(gr_text "74"
+			(at 92.5 103.85 0)
+			(layer "Dwgs.User")
+			(effects
+				(font
+					(size 1 1)
+					(thickness 0.15)
+				)
+			)
+		)
+	)
+	(dimension
+		(type orthogonal)
+		(layer "Dwgs.User")
+		(pts
+			(xy 55.5 22.5) (xy 55.5 96.5)
+		)
+		(height -9)
+		(orientation 1)
+		(format
+			(prefix "")
+			(suffix "")
+			(units 3)
+			(units_format 0)
+			(precision 4)
+			(suppress_zeroes yes)
+		)
+		(style
+			(thickness 0.1)
+			(arrow_length 1.27)
+			(text_position_mode 0)
+			(arrow_direction outward)
+			(extension_height 0.58642)
+			(extension_offset 0.5)
+			(keep_text_aligned yes)
+		)
+		(gr_text "74"
+			(at 45.35 59.5 90)
+			(layer "Dwgs.User")
+			(effects
+				(font
+					(size 1 1)
+					(thickness 0.15)
+				)
+			)
+		)
+	)
 	(segment
 		(start 114 98.4)
@@
 	)
 	(segment
-		(start 121.5 54)
-		(end 116 59.5)
-		(width 0.2)
-		(layer "F.Cu")
-		(net "+5V")
-	)
-	(segment
 		(start 80 41.16)
 		(end 69.66 41.16)
@@
 	)
 	(segment
+		(start 121.5 54)
+		(end 115.5 60)
+		(width 0.2)
+		(layer "F.Cu")
+		(net "+5V")
+	)
+	(segment
 		(start 98 57)
 		(end 97.8 56.8)
@@
 	)
 	(segment
+		(start 115.5 94.45)
+		(end 116 94.95)
+		(width 0.2)
+		(layer "F.Cu")
+		(net "+5V")
+	)
+	(segment
 		(start 116 94.95)
 		(end 116 96.4)
@@
 	)
 	(segment
+		(start 115.5 60)
+		(end 115.5 94.45)
+		(width 0.2)
+		(layer "F.Cu")
+		(net "+5V")
+	)
+	(segment
 		(start 93 75)
 		(end 95.5 75)
@@
 	)
 	(segment
-		(start 116 59.5)
-		(end 116 94.95)
-		(width 0.2)
-		(layer "F.Cu")
-		(net "+5V")
-	)
-	(segment
 		(start 117 22.5)
 		(end 124.08 29.58)
@@
 	)
 	(segment
+		(start 83.2175 34.5)
+		(end 83 34.2825)
+		(width 0.2)
+		(layer "F.Cu")
+		(net "GND")
+	)
+	(segment
 		(start 106.5 92.5)
 		(end 106.5 93.5)
@@
 	)
 	(segment
-		(start 83.2175 34.5)
-		(end 87 34.5)
-		(width 0.2)
-		(layer "F.Cu")
-		(net "GND")
-	)
-	(segment
 		(start 105.5 33.511)
 		(end 105.5 33.036)
@@
 	)
 	(segment
-		(start 83 34.2825)
-		(end 83.2175 34.5)
-		(width 0.2)
-		(layer "F.Cu")
-		(net "GND")
-	)
-	(segment
 		(start 84 95.5)
 		(end 84.5 95)
@@
 	)
 	(segment
+		(start 86.5 34.5)
+		(end 83.2175 34.5)
+		(width 0.2)
+		(layer "F.Cu")
+		(net "GND")
+	)
+	(segment
 		(start 66.5 31.511)
 		(end 66.5 37.511)
@@
 	)
 	(segment
+		(start 87.5 33.5)
+		(end 86.5 34.5)
+		(width 0.2)
+		(layer "F.Cu")
+		(net "GND")
+	)
+	(segment
 		(start 100.5 84)
 		(end 100.775 83.725)
@@
 	)
 	(via
-		(at 87 34.5)
+		(at 87.5 33.5)
 		(size 0.508)
 		(drill 0.3048)
@@
 	)
 	(segment
-		(start 88.284772 34.5)
-		(end 87 34.5)
-		(width 0.2)
-		(layer "B.Cu")
-		(net "GND")
-	)
-	(segment
-		(start 108.5 44.96)
-		(end 107.04 43.5)
-		(width 0.2)
-		(layer "B.Cu")
-		(net "GND")
-	)
-	(segment
 		(start 88.6435 67.9125)
 		(end 89.7935 66.7625)
@@
 	)
 	(segment
-		(start 107.04 43.5)
-		(end 103 43.5)
-		(width 0.2)
-		(layer "B.Cu")
-		(net "GND")
-	)
-	(segment
 		(start 92.1935 66.7625)
 		(end 90.9935 66.7625)
@@
 	)
 	(segment
-		(start 107.04 43.5)
-		(end 105.5 41.96)
-		(width 0.2)
-		(layer "B.Cu")
-		(net "GND")
-	)
-	(segment
 		(start 95.9635 67.9125)
 		(end 95.7435 67.9125)
@@
 	)
 	(segment
-		(start 103 43.5)
-		(end 101.5 42)
-		(width 0.2)
-		(layer "B.Cu")
-		(net "GND")
-	)
-	(segment
 		(start 114.05 51.5)
 		(end 114 51.5)
@@
 	)
 	(segment
-		(start 95.784772 42)
-		(end 88.284772 34.5)
-		(width 0.2)
-		(layer "B.Cu")
-		(net "GND")
-	)
-	(segment
 		(start 90.9935 71.0625)
 		(end 89.7935 71.0625)
@@
 	)
 	(segment
-		(start 101.5 42)
-		(end 95.784772 42)
-		(width 0.2)
-		(layer "B.Cu")
-		(net "GND")
-	)
-	(segment
-		(start 105.5 41.96)
-		(end 105.5 35.5)
-		(width 0.2)
-		(layer "B.Cu")
-		(net "GND")
-	)
-	(segment
 		(start 95.7935 68.0825)
 		(end 95.9635 67.9125)
@@
 	)
 	(segment
+		(start 109.672189 42.458642)
+		(end 109.672189 46.132189)
+		(width 0.2)
+		(layer "F.Cu")
+		(net "/GPIO14{slash}TXD0")
+	)
+	(segment
 		(start 60.5 61.5)
 		(end 60.58 61.42)
@@
 	)
 	(segment
-		(start 60.58 61.42)
-		(end 60.58 57)
+		(start 109.672189 46.132189)
+		(end 111.04 47.5)
 		(width 0.2)
 		(layer "F.Cu")
@@
 	)
 	(segment
-		(start 111.04 47.5)
-		(end 109.672189 46.132189)
+		(start 60.58 61.42)
+		(end 60.58 57)
 		(width 0.2)
 		(layer "F.Cu")
@@
 	)
 	(segment
-		(start 109.672189 46.132189)
+		(start 109.5 42.286453)
 		(end 109.672189 42.458642)
 		(width 0.2)
@@
 	)
 	(via
-		(at 109.672189 42.458642)
+		(at 109.5 42.286453)
 		(size 0.508)
 		(drill 0.3048)
@@
 	)
 	(segment
-		(start 109.672189 42.458642)
-		(end 109.5 42.286453)
-		(width 0.2)
-		(layer "B.Cu")
-		(net "/GPIO14{slash}TXD0")
-	)
-	(segment
 		(start 62 63)
 		(end 60.5 61.5)
@@
 	)
 	(segment
-		(start 109 35.5)
-		(end 108.5 35)
+		(start 107.171051 42)
+		(end 107.171051 46.171051)
 		(width 0.2)
 		(layer "F.Cu")
@@
 	)
 	(segment
-		(start 58.04 57)
-		(end 58.04 60.04)
+		(start 109 35.5)
+		(end 108.5 35)
 		(width 0.2)
 		(layer "F.Cu")
@@
 	)
 	(segment
-		(start 107.171051 46.171051)
-		(end 107.171051 42.458642)
+		(start 58.04 57)
+		(end 58.04 60.04)
 		(width 0.2)
 		(layer "F.Cu")
@@
 	)
 	(segment
-		(start 108.5 47.5)
-		(end 107.171051 46.171051)
+		(start 108.5 35)
+		(end 108.5 33.511)
 		(width 0.2)
 		(layer "F.Cu")
@@
 	)
 	(segment
-		(start 108.5 35)
-		(end 108.5 33.511)
+		(start 107.171051 46.171051)
+		(end 108.5 47.5)
 		(width 0.2)
 		(layer "F.Cu")
@@
 	)
 	(via
-		(at 107.171051 42.458642)
+		(at 107.171051 42)
 		(size 0.508)
 		(drill 0.3048)
@@
 	)
 	(segment
+		(start 107.171051 37.828949)
+		(end 109 36)
+		(width 0.2)
+		(layer "B.Cu")
+		(net "/GPIO15{slash}RXD0")
+	)
+	(segment
 		(start 95.5 62.5)
 		(end 108.5 49.5)
@@
 	)
 	(segment
-		(start 107.171051 37.828949)
-		(end 109 36)
+		(start 107.171051 42)
+		(end 107.171051 37.828949)
 		(width 0.2)
 		(layer "B.Cu")
@@
 		(width 0.2)
 		(layer "B.Cu")
-		(net "/GPIO15{slash}RXD0")
-	)
-	(segment
-		(start 107.171051 42.458642)
-		(end 107.171051 37.828949)
-		(width 0.2)
-		(layer "B.Cu")

Commit message: Updated Throughhole
Routing:
- net GND: track 173.7 -> 173.1 mm
Changed lines of the file:
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@@
 		)
 		(embedded_fonts no)
-		(model "${KICAD6_3DMODEL_DIR}/Package_LGA.3dshapes/Bosch_LGA-8_2.5x2.5mm_P0.65mm_ClockwisePinNumbering.wrl"
+		(model "${KICAD10_3DMODEL_DIR}/Package_LGA.3dshapes/Bosch_LGA-8_2.5x2.5mm_P0.65mm_ClockwisePinNumbering.step"
 			(offset
 				(xyz 0.01500000025 -0.03500000059 0)
@@
 		)
 		(embedded_fonts no)
-		(model "${KICAD6_3DMODEL_DIR}/Package_LGA.3dshapes/Bosch_LGA-8_2.5x2.5mm_P0.65mm_ClockwisePinNumbering.wrl"
+		(model "${KICAD10_3DMODEL_DIR}/Package_LGA.3dshapes/Bosch_LGA-8_2.5x2.5mm_P0.65mm_ClockwisePinNumbering.step"
 			(offset
 				(xyz 0.01500000025 -0.03500000059 0)
@@
 	)
 	(segment
-		(start 114.05 47.97)
-		(end 113.58 47.5)
-		(width 0.2)
-		(layer "F.Cu")
-		(net "GND")
-	)
-	(segment
 		(start 98.975 94.475)
 		(end 98.975 94.975)
@@
 	(via
 		(at 93.869707 68.846765)
-		(size 0.508)
-		(drill 0.3048)
+		(size 0.458)
+		(drill 0.2548)
 		(layers "F.Cu" "B.Cu")
 		(net "/5V_BUS_USB")
@@
 	)
 	(segment
-		(start 90.9435 68.863511)
-		(end 90.9435 69.7425)
+		(start 93.4435 68.0825)
+		(end 93.4435 69.272972)
 		(width 0.2)
 		(layer "B.Cu")
@@
 	)
 	(segment
-		(start 90.9435 68.0825)
-		(end 90.9435 68.863511)
+		(start 90.9435 68.863511)
+		(end 90.9435 69.7425)
 		(width 0.2)
 		(layer "B.Cu")
@@
 	)
 	(segment
-		(start 93.4435 68.0825)
-		(end 93.4435 68.420558)
+		(start 90.9435 68.0825)
+		(end 90.9435 68.863511)
 		(width 0.2)
 		(layer "B.Cu")
@@
 		(end 93.869707 68.846765)
 		(width 0.254)
-		(layer "B.Cu")
-		(net "/5V_BUS_USB")
-	)
-	(segment
-		(start 93.4435 68.420558)
-		(end 93.869707 68.846765)
-		(width 0.254)
