File: kiCad/dreamV3_0/Dream_V3.kicad_pcb (KiCad board)
At the start: 2 copper layers, 80 x 80 mm, 44 parts, among them IC1 TGS2611-C00, J1 GPIO, J11 10132328-10011LF, J2 Qwiic_Vertical, J3 679305124022, J4 Qwiic_Vertical, J5 M20-7830542, J6 Qwiic_Vertical, J7 5013310607, J8 Qwiic_4pin_Vertical, J9 Qwiic_Vertical, Q1 BSS138, U1 AP2112K-3.3, U2 BME280, U3 INA219BxDCN, U5 BME280

Commit message: final dreamV3
Parts:
- S1: value OS102011MA1QN1 -> NK236
Connections:
- J1 pad : +3V3 -> (no net)
- J1 pad 27: /ID_SDA -> /PI10/RXD1
- J1 pad 28: /ID_SCL -> /PI9/TXD1
- J6 pad 2: +3V3 -> +5V
- J6 pad 3: /GPIO14/TXD0 -> /PI9/TXD1
- J6 pad 4: /GPIO15/RXD0 -> /PI10/RXD1
- S1 pad 1: /5V_BUS_USB -> +5V
- S1 pad 2: +5V -> /5V_BUS_USB
- U1 pad en: +3V3 -> (no net)
- U3 pad 2: INA- -> Net-(U3-IN-)
Routing:
- net /PI9/TXD1: track 0.00 -> 35.8 mm, vias 0 -> 1
- net /PI10/RXD1: track 0.00 -> 32.5 mm, vias 0 -> 1
- net /GPIO15/RXD0: track 77.4 -> 61.9 mm, vias 3 -> 1
- net /GPIO14/TXD0: track 77.6 -> 62.1 mm, vias 3 -> 1
- net +3V3: track 190.7 -> 175.8 mm
- net +5V: track 285.5 -> 300.1 mm
- net GND: track 173.1 -> 174.4 mm

Commit message: final dreamV3
Parts:
- moved J6 14.5 mm to (92.5, 32.0)
Connections:
- J6 pad 2: +5V -> +3V3
- S1 pad 1: +5V -> /5V_BUS_USB
- S1 pad 2: /5V_BUS_USB -> +5V
Routing:
- net /PI9/TXD1: track 35.8 -> 20.7 mm
- net /PI10/RXD1: track 32.5 -> 17.5 mm
- net +5V: track 300.1 -> 291.4 mm
- net +3V3: track 175.8 -> 181.6 mm
- net GND: track 174.4 -> 175.1 mm, vias 9 -> 8
- net /5V_BUS_USB: track 76.7 -> 76.2 mm
Other:
- board text added: "All supply levels are 5V unless otherwise indicated"
- board text removed: "- - -"
- board text removed: "5V"

Commit message: Updated PCB
Connections:
- J6 pad 2: +3V3 -> +5V
- S1 pad 1: /5V_BUS_USB -> +5V
- S1 pad 2: +5V -> /5V_BUS_USB
Routing:
- net +5V: track 291.4 -> 299.1 mm
- net +3V3: track 181.6 -> 175.2 mm
Changed lines of the file:
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@@
 		(capping no)
 		(filling no)
-		(zone_defaults)
 		(pcbplotparams
 			(layerselection 0x00000000_00000000_55555555_5755f5ff)
@@
 			(size 0.6 1.55)
 			(layers "F.Cu" "F.Mask" "F.Paste")
-			(net "+3V3")
+			(net "+5V")
 			(pinfunction "Pin_2_2")
 			(pintype "passive")
@@
 			(layers "*.Cu" "*.Mask")
 			(remove_unused_layers no)
-			(net "/5V_BUS_USB")
+			(net "+5V")
 			(pintype "passive")
 		)
@@
 			(layers "*.Cu" "*.Mask")
 			(remove_unused_layers no)
-			(net "+5V")
+			(net "/5V_BUS_USB")
 			(pintype "passive")
 		)
@@
 	)
 	(segment
-		(start 105.5 33.781074)
-		(end 105.5 41.16)
-		(width 0.25)
-		(layer "F.Cu")
-		(net "+5V")
-	)
-	(segment
 		(start 124.08 40.5)
 		(end 124.08 42.08)
@@
 	)
 	(segment
+		(start 92 33.036)
+		(end 92.566252 32.469748)
+		(width 0.2)
+		(layer "F.Cu")
+		(net "+5V")
+	)
+	(segment
 		(start 115.95 47.67)
 		(end 116.12 47.5)
@@
 	)
 	(segment
+		(start 92 33.511)
+		(end 92 33.036)
+		(width 0.2)
+		(layer "F.Cu")
+		(net "+5V")
+	)
+	(segment
 		(start 99.5 57)
 		(end 98 57)
@@
 	)
 	(segment
+		(start 97.643972 32.469748)
+		(end 97.643972 41.016028)
+		(width 0.2)
+		(layer "F.Cu")
+		(net "+5V")
+	)
+	(segment
 		(start 99.0875 69.4125)
 		(end 99.817621 69.4125)
@@
 	)
 	(segment
+		(start 97.643972 41.016028)
+		(end 97.5 41.16)
+		(width 0.2)
+		(layer "F.Cu")
+		(net "+5V")
+	)
+	(segment
 		(start 115.5 94.45)
 		(end 116 94.95)
@@
 	)
 	(segment
+		(start 80 41.16)
+		(end 97.5 41.16)
+		(width 0.5)
+		(layer "F.Cu")
+		(net "+5V")
+	)
+	(segment
 		(start 116 94.95)
 		(end 116 96.4)
@@
 	)
 	(segment
+		(start 92.566252 32.469748)
+		(end 97.643972 32.469748)
+		(width 0.2)
+		(layer "F.Cu")
+		(net "+5V")
+	)
+	(segment
 		(start 117 22.5)
 		(end 124.08 29.58)
@@
 	)
 	(segment
-		(start 80 41.16)
+		(start 97.5 41.16)
 		(end 105.5 41.16)
 		(width 0.5)
@@
 	)
 	(segment
-		(start 92 33.036)
-		(end 92.566252 32.469748)
-		(width 0.2)
-		(layer "F.Cu")
-		(net "+3V3")
-	)
-	(segment
 		(start 104 80)
 		(end 102 82)
@@
 	)
 	(segment
-		(start 92.566252 32.469748)
-		(end 95.066252 32.469748)
-		(width 0.2)
-		(layer "F.Cu")
-		(net "+3V3")
-	)
-	(segment
 		(start 87.5 73.5)
 		(end 87.5 75)
@@
 	)
 	(segment
-		(start 92 33.511)
-		(end 92 33.036)
-		(width 0.2)
-		(layer "F.Cu")
-		(net "+3V3")
-	)
-	(segment
 		(start 103.2 85.2)
 		(end 102.7 85.2)
 		(width 0.2)
 		(layer "F.Cu")
-		(net "+3V3")
-	)
-	(segment
-		(start 95.066252 32.469748)
-		(end 97.643972 32.469748)
-		(width 0.2)
-		(layer "F.Cu")

Commit message: ACTUAL final DreamV3
Parts:
- added Q2: BSS138, PCM_SparkFun-Semiconductor-Standard:SOT-363, F.Cu at (103.0, 86.0)
- IC1: footprint TGS2611_clean:TGS2611C00 -> tgs2611:tgs2611c00
- R3: value 10k -> 2k
- moved R10 4.25 mm to (100.5, 90.0), turned to 90 degrees
- moved R13 3.42 mm to (107.5, 86.0)
- moved IC1 2.55 mm to (91.0, 89.5)
- moved JP4 1.50 mm to (103.0, 90.5)
- moved R9 0.50 mm to (81.5, 90.0)
- turned U2 to -90 degrees
Connections:
- J1 pad : (no net) -> +3V3
- R5 pad 1: /GPIO23/SDA4 -> /GPIO2/SDA1
- R5 pad 3: /GPIO24/SCL4 -> /GPIO3/SCL1
- S1 pad 1: +5V -> /5V_BUS_USB
- S1 pad 2: /5V_BUS_USB -> +5V
- U1 pad en: (no net) -> +3V3
- U3 pad 2: Net-(U3-IN-) -> INA-
Routing:
- net /GPIO3/SCL1: track 60.0 -> 73.2 mm, vias 3 -> 4
- net /GPIO2/SDA1: track 64.8 -> 77.6 mm, vias 3 -> 4
- net /BME_SCL2: track 9.60 -> 22.1 mm, vias 0 -> 2
- net /BME_SDA2: track 13.6 -> 19.0 mm, vias 0 -> 2
- net /GPIO23/SDA4: track 79.0 -> 83.4 mm, vias 4 -> 7
- net /GPIO24/SCL4: track 82.8 -> 79.3 mm
- net GND: track 175.1 -> 171.8 mm
- net BME_3V3: track 70.1 -> 72.6 mm
- net +5V: track 299.1 -> 297.0 mm
- net /BME_ADD_2: track 4.38 -> 5.98 mm
- net +3V3: track 175.2 -> 176.4 mm, vias 5 -> 7
- net /INA+: track 15.1 -> 14.0 mm
- net /GPIO27/SDA3: track 99.2 -> 98.6 mm
Other:
- board text added: "REQUIRES ORANGE PI"
