File: kiCad/dreamV3_0/Dream_V3.kicad_pcb (KiCad board)
At the start: 2 copper layers, 80 x 80 mm, 45 parts, among them IC1 TGS2611-C00, J1 GPIO, J11 10132328-10011LF, J2 Qwiic_Vertical, J3 679305124022, J4 Qwiic_Vertical, J5 M20-7830542, J6 Qwiic_Vertical, J7 5013310607, J8 Qwiic_4pin_Vertical, J9 Qwiic_Vertical, Q1 BSS138, Q2 BSS138, U1 AP2112K-3.3, U2 BME280, U3 INA219BxDCN, U5 BME280

Commit message: ACTUAL final dreamV3
Routing:
- net /BME_SDA2: track 19.0 -> 18.1 mm
- net +5V: track 297.0 -> 296.1 mm

Commit message: ACTUAL final dreamV3
Parts:
- C7: value EEV107M010S9GAA -> 100UF
- R4: value R_US -> 0.1
- R6: value RC0603FR-075K1L -> 5.1k
- R8: value RC0603FR-07330RL -> 330
Changed lines of the file:
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@@
 		(capping no)
 		(filling no)
+		(zone_defaults)
 		(pcbplotparams
 			(layerselection 0x00000000_00000000_55555555_5755f5ff)
@@
 			(at 1.25 -4.4 0)
 			(layer "F.SilkS")
+			(hide yes)
 			(effects
 				(font
@@
 			)
 		)
-		(property "Value" "EEV107M010S9GAA"
+		(property "Value" "100UF"
 			(at 1.25 4.4 0)
 			(layer "F.Fab")
@@
 			)
 		)
+		(property "Vendor" "https://www.digikey.com/en/products/detail/diodes-incorporated/AP2112K-3-3TRG1/4470746?s=N4IgTCBcDaIIIAUwEZlgNIFoDMA6bIAugL5A"
+			(at 0 0 270)
+			(unlocked yes)
+			(layer "F.Fab")
+			(hide yes)
+			(effects
+				(font
+					(size 1 1)
+					(thickness 0.15)
+				)
+			)
+		)
 		(property ki_fp_filters "SOT?23?5*")
 		(sheetname "/")
@@
 			(at 0.015 -2.465 90)
 			(layer "F.SilkS")
+			(hide yes)
 			(effects
 				(font
@@
 			)
 		)
+		(property "Vendor" "https://www.digikey.com/en/products/detail/bosch-sensortec/BME280/6136306"
+			(at 0 0 90)
+			(unlocked yes)
+			(layer "F.Fab")
+			(hide yes)
+			(effects
+				(font
+					(size 1 1)
+					(thickness 0.15)
+				)
+			)
+		)
 		(property ki_fp_filters "*LGA*2.5x2.5mm*P0.65mm*Clockwise*")
 		(sheetname "/")
@@
 			(at -0.26 -1.1 90)
 			(layer "F.SilkS")
+			(hide yes)
 			(effects
 				(font
 					(size 0.393701 0.393701)
-					(thickness 0.15)
+					(thickness 0.058425)
 				)
 			)
 		)
-		(property "Value" "RC0603FR-075K1L"
+		(property "Value" "5.1k"
 			(at 0.265 1.5 90)
 			(layer "F.Fab")
@@
 				(font
 					(size 0.393701 0.393701)
-					(thickness 0.15)
+					(thickness 0.098425)
 				)
 			)
@@
 			(at 0 -1.17 0)
 			(layer "F.SilkS")
+			(hide yes)
 			(effects
 				(font
@@
 			(at -0.1 -1.43 90)
 			(layer "F.SilkS")
+			(hide yes)
 			(effects
 				(font
@@
 			)
 		)
-		(property "Description" ""
+		(property "Description" "RES 5.1K OHM 1% 1/10W 0603"
 			(at 0 0 90)
 			(layer "F.Fab")
@@
 				(font
 					(size 0.393701 0.393701)
-					(thickness 0.15)
+					(thickness 0.038425)
 				)
 			)
 		)
-		(property "Value" "RC0603FR-07330RL"
+		(property "Value" "330"
 			(at 1.49 1.1 0)
 			(layer "F.Fab")
+			(hide yes)
 			(effects
 				(font
 					(size 0.393701 0.393701)
-					(thickness 0.15)
+					(thickness 0.098425)
 				)
 			)
@@
 			)
 		)
+		(property "Vendor" "https://www.digikey.com/en/products/detail/taiyo-yuden/TMK212BBJ106KG-T/2714163"
+			(at 0 0 90)
+			(unlocked yes)
+			(layer "F.Fab")
+			(hide yes)
+			(effects
+				(font
+					(size 1 1)
+					(thickness 0.15)
+				)
+			)
+		)
 		(property ki_fp_filters "C_*")
 		(sheetname "/")
@@
 			)
 		)
+		(property "Vendor" "https://www.digikey.com/en/products/detail/bourns-inc/CAT16-1002F4LF/3593233?s=N4IgjCBcodIMZQGYEMA2BnApgGhAeygG0QB2AZgBYAGckAXTwAcAXKEAZRYCcBLAOwDmIAL546cRJFSZcBYuDDkIjEK3Zc%2BQ0XjAA2KKCkzseQpBIAOcqQBMthszaROPAcLEhbyyoYTJ0U3kLL1p9Ukc1Z1ctDzwAWlgjANkzBTAwSwZPeIdJKB4AVzlzEgBWEDwATmyEiWTIIpL06lqQeIN8xu5itJC6PF88B3oc3y6TZpD7UlpK8EsyvRURVaA"
+			(at 0 0 270)
+			(unlocked yes)
+			(layer "F.Fab")
+			(hide yes)
+			(effects
+				(font
+					(size 1 1)
+					(thickness 0.15)
+				)
+			)
+		)
 		(property ki_fp_filters "R_*")
 		(sheetname "/")
@@
 			)
 		)
+		(property "Vendor" "https://www.digikey.com/en/products/detail/bourns-inc/CAT16-1002F4LF/3593233?s=N4IgjCBcodIMZQGYEMA2BnApgGhAeygG0QB2AZgBYAGckAXTwAcAXKEAZRYCcBLAOwDmIAL546cRJFSZcBYuDDkIjEK3Zc%2BQ0XjAA2KKCkzseQpBIAOcqQBMthszaROPAcLEhbyyoYTJ0U3kLL1p9Ukc1Z1ctDzwAWlgjANkzBTAwSwZPeIdJKB4AVzlzEgBWEDwATmyEiWTIIpL06lqQeIN8xu5itJC6PF88B3oc3y6TZpD7UlpK8EsyvRURVaA"
+			(at 0 0 0)
+			(unlocked yes)
+			(layer "F.Fab")
+			(hide yes)
+			(effects
+				(font
+					(size 1 1)
+					(thickness 0.15)
+				)
+			)
+		)
 		(property ki_fp_filters "R_*")
 		(sheetname "/")
@@
 			)
 		)
-		(property "Value" "R_US"
+		(property "Value" "0.1"
 			(at 0 1.65 90)
 			(layer "F.Fab")
@@
 			)
 		)
-		(property "Datasheet" ""
+		(property "Datasheet" "https://www.yageogroup.com/content/Resource%20Library/Datasheet/PYU-PT-GROUP_521_ROHS_L.pdf"
 			(at 0 0 90)
 			(layer "F.Fab")
@@
 			)
 		)
-		(property "Description" "Resistor, US symbol"
+		(property "Description" "RES 0.1 OHM 1% 1W 2512"
 			(at 0 0 90)
 			(layer "F.Fab")
@@
 			)
 		)
+		(property "Vendor" "https://www.digikey.com/en/products/detail/yageo/PT2512FK-070R1L/2178346?s=N4IgTCBcDaIAoBUwFYCMYBiBpAtABgHY8AlVAGRAF0BfIA"
+			(at 0 0 0)
+			(unlocked yes)
+			(layer "F.Fab")
+			(hide yes)
+			(effects
+				(font
+					(size 1 1)
+					(thickness 0.15)
+				)
+			)
+		)
 		(property ki_fp_filters "R_*")
 		(sheetname "/")
@@
 			)
 		)
+		(property "Vendor" "https://www.digikey.com/en/products/detail/bourns-inc/CAT16-1002F4LF/3593233?s=N4IgjCBcodIMZQGYEMA2BnApgGhAeygG0QB2AZgBYAGckAXTwAcAXKEAZRYCcBLAOwDmIAL546cRJFSZcBYuDDkIjEK3Zc%2BQ0XjAA2KKCkzseQpBIAOcqQBMthszaROPAcLEhbyyoYTJ0U3kLL1p9Ukc1Z1ctDzwAWlgjANkzBTAwSwZPeIdJKB4AVzlzEgBWEDwATmyEiWTIIpL06lqQeIN8xu5itJC6PF88B3oc3y6TZpD7UlpK8EsyvRURVaA"
+			(at 0 0 0)
+			(unlocked yes)
+			(layer "F.Fab")
+			(hide yes)
+			(effects
+				(font
+					(size 1 1)
+					(thickness 0.15)
+				)
+			)
+		)
 		(property ki_fp_filters "R_*")
 		(sheetname "/")
@@
 			)
 		)
+		(property "Vendor" "https://www.digikey.com/en/products/detail/bourns-inc/CAT16-1002F4LF/3593233?s=N4IgjCBcodIMZQGYEMA2BnApgGhAeygG0QB2AZgBYAGckAXTwAcAXKEAZRYCcBLAOwDmIAL546cRJFSZcBYuDDkIjEK3Zc%2BQ0XjAA2KKCkzseQpBIAOcqQBMthszaROPAcLEhbyyoYTJ0U3kLL1p9Ukc1Z1ctDzwAWlgjANkzBTAwSwZPeIdJKB4AVzlzEgBWEDwATmyEiWTIIpL06lqQeIN8xu5itJC6PF88B3oc3y6TZpD7UlpK8EsyvRURVaA"
+			(at 0 0 0)
+			(unlocked yes)
+			(layer "F.Fab")
+			(hide yes)
+			(effects
+				(font
+					(size 1 1)
+					(thickness 0.15)
+				)
+			)
+		)
 		(property ki_fp_filters "R_*")
 		(sheetname "/")
@@
 			(at 0.015 -2.465 90)
 			(layer "F.SilkS")
+			(hide yes)
 			(effects
 				(font
@@
 			)
 		)
+		(property "Vendor" "https://www.digikey.com/en/products/detail/bosch-sensortec/BME280/6136306"
+			(at 0 0 270)
+			(unlocked yes)
+			(layer "F.Fab")
+			(hide yes)
+			(effects
+				(font
+					(size 1 1)
+					(thickness 0.15)
+				)
+			)
+		)
 		(property ki_fp_filters "*LGA*2.5x2.5mm*P0.65mm*Clockwise*")
 		(sheetname "/")
@@
 			(at 0 -1.17 0)
 			(layer "F.SilkS")
+			(hide yes)
 			(effects
 				(font
@@
 			)
 		)
+		(property "Vendor" "https://www.digikey.com/en/products/detail/texas-instruments/INA219BIDCNT/2426056"
+			(at 0 0 90)
+			(unlocked yes)
+			(layer "F.Fab")
+			(hide yes)
+			(effects
+				(font
+					(size 1 1)
+					(thickness 0.15)
+				)
+			)
+		)
 		(property ki_fp_filters "SOT?23*")
 		(sheetname "/")
@@
 			)
 		)
-		(property "Datasheet" ""
+		(property "Datasheet" "https://mm.digikey.com/Volume0/opasdata/d220001/medias/docus/6129/ssw-1xx-xx-xxx-x-xx-xxx-xx-mkt.pdf"
 			(at 0 0 90)
 			(layer "B.Fab")
@@
 					(thickness 0.15)
 				)
+				(justify mirror)
+			)
+		)
+		(property "Vendor" "https://www.digikey.com/en/products/detail/samtec-inc/SSW-120-02-G-D/1112335"
+			(at 0 0 0)
+			(unlocked yes)
+			(layer "B.Fab")
+			(hide yes)
+			(effects
+				(font
+					(size 1 1)
+					(thickness 0.15)
+				)

Commit message: ACTUAL ACTUAL final dreamV3
Parts:
- IC1: value TGS2611-C00 -> SR-6
Routing:
- net BME_3V3: track 72.6 -> 78.8 mm
- net /BME_ADD_2: track 5.98 -> 11.0 mm, vias 0 -> 2
- net GND: track 171.8 -> 168.3 mm
Changed lines of the file:
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@@
 			)
 		)
-		(property "Value" "TGS2611-C00"
+		(property "Value" "SR-6"
 			(at 0.5 5.5 0)
 			(unlocked yes)
@@
 			)
 		)
-		(property "Description" "Figaro TGS2611-C00 Methane Gas Sensor"
+		(property "Description" "SR-6 Sensor Socket"
 			(at 0 0 0)
 			(unlocked yes)
@@
 	)
 	(segment
-		(start 106.5 92.5)
-		(end 106.5 93.5)
-		(width 0.2)
-		(layer "F.Cu")
-		(net "GND")
-	)
-	(segment
 		(start 102.317621 73.732379)
 		(end 102.05 74)
@@
 	)
 	(segment
-		(start 103 90.0936)
-		(end 104.0936 89)
-		(width 0.2)
-		(layer "F.Cu")
-		(net "GND")
-	)
-	(segment
 		(start 90.5 75.6)
 		(end 91.4 75.6)
@@
 	)
 	(segment
-		(start 106.5 93.5)
-		(end 105 95)
-		(width 0.2)
-		(layer "F.Cu")
-		(net "GND")
-	)
-	(segment
-		(start 104.0936 89)
-		(end 104.5 89)
-		(width 0.2)
-		(layer "F.Cu")
-		(net "GND")
-	)
-	(segment
 		(start 86 53.265)
 		(end 83.785 53.265)
@@
 	)
 	(segment
+		(start 103.0936 90)
+		(end 103 90.0936)
+		(width 0.2)
+		(layer "F.Cu")
+		(net "GND")
+	)
+	(segment
 		(start 100.05 92.55)
 		(end 99.5 92)
@@
 	)
 	(segment
+		(start 104.5 90)
+		(end 103.0936 90)
+		(width 0.2)
+		(layer "F.Cu")
+		(net "GND")
+	)
+	(segment
 		(start 88.5 53.175)
 		(end 88.5 52.9)
@@
 	)
 	(via
-		(at 104.5 89)
+		(at 104.5 90)
 		(size 0.6)
 		(drill 0.3)
@@
 	)
 	(segment
+		(start 107.409383 87.090617)
+		(end 107.409383 87.473481)
+		(width 0.2)
+		(layer "F.Cu")
+		(net "BME_3V3")
+	)
+	(segment
 		(start 79.8 87.3)
 		(end 79.8 86.5)
@@
 	)
 	(segment
+		(start 107.409383 87.473481)
+		(end 106.882864 88)
+		(width 0.2)
+		(layer "F.Cu")
+		(net "BME_3V3")
+	)
+	(segment
 		(start 85.179551 87.320449)
 		(end 85.5 87)
@@
 	)
 	(segment
+		(start 106.882864 88)
+		(end 106.116154 88)
+		(width 0.2)
+		(layer "F.Cu")
+		(net "BME_3V3")
+	)
+	(segment
 		(start 100.529004 89.13907)
 		(end 100.143329 89.13907)
@@
 	)
 	(segment
+		(start 104.116154 86)
+		(end 103.95 86)
+		(width 0.2)
+		(layer "F.Cu")
+		(net "BME_3V3")
+	)
+	(segment
 		(start 101 93.2)
 		(end 101.312856 93.2)
@@
 	)
 	(segment
+		(start 106.116154 88)
+		(end 104.116154 86)
+		(width 0.2)
+		(layer "F.Cu")
+		(net "BME_3V3")
+	)
+	(segment
 		(start 86 87)
 		(end 87.05 85.95)
@@
 	)
 	(segment
+		(start 108.1 86.4)
+		(end 107.409383 87.090617)
+		(width 0.2)
+		(layer "F.Cu")
+		(net "BME_3V3")
+	)
+	(segment
 		(start 91 81.5875)
 		(end 91.95 80.6375)
@@
 	)
 	(segment
+		(start 108.4 86.4)
+		(end 108.1 86.4)
+		(width 0.2)
+		(layer "F.Cu")
+		(net "BME_3V3")
+	)
+	(segment
 		(start 92.85 93.85)
 		(end 91 92)
@@
 		(start 118.66 44.96)
 		(end 119.775057 44.96)
-		(width 0.4064)
+		(width 0.5)
 		(layer "F.Cu")
 		(net "+3V3")
@@
 		(start 119.775057 44.96)
 		(end 122.829384 41.905673)
-		(width 0.4064)
+		(width 0.5)
 		(layer "F.Cu")
 		(net "+3V3")
@@
 	)
 	(segment
+		(start 102 95.5)
+		(end 103 94.5)
+		(width 0.2)
+		(layer "F.Cu")
+		(net "/BME_ADD_2")
+	)
+	(segment
 		(start 99.95 95.5)
 		(end 102 95.5)
@@
 	)
 	(segment
+		(start 103 92)
+		(end 103 90.9064)
+		(width 0.2)
+		(layer "F.Cu")
+		(net "/BME_ADD_2")
+	)
+	(segment
 		(start 98.95 94.5)
 		(end 99.95 95.5)
@@
 		(net "/BME_ADD_2")
 	)
+	(via
+		(at 103 94.5)
+		(size 0.6)
+		(drill 0.3)
+		(layers "F.Cu" "B.Cu")
+		(net "/BME_ADD_2")
+	)
+	(via
+		(at 103 92)
+		(size 0.6)
+		(drill 0.3)
+		(layers "F.Cu" "B.Cu")
+		(net "/BME_ADD_2")
+	)
+	(segment
+		(start 103 92)
+		(end 103 94.5)
+		(width 0.2)
+		(layer "B.Cu")
+		(net "/BME_ADD_2")
+	)
