File: kiCad/dreamV3_0/Dream_V3.kicad_pcb (KiCad board)
At the start: 2 copper layers, 80 x 80 mm, 45 parts, among them IC1 SR-6, J1 GPIO, J11 10132328-10011LF, J2 Qwiic_Vertical, J3 679305124022, J4 Qwiic_Vertical, J5 M20-7830542, J6 Qwiic_Vertical, J7 5013310607, J8 Qwiic_4pin_Vertical, J9 Qwiic_Vertical, Q1 BSS138, Q2 BSS138, U1 AP2112K-3.3, U2 BME280, U3 INA219BxDCN, U5 BME280

Commit message: update switch properties
Parts:
- S1: value NK236 -> EG1224
