File: kiCad/dreamV3_0/Dream_V3.kicad_sch (KiCad schematic)
At the start: 42 parts, among them IC1 TGS2611-C00, J1 GPIO, J11 10132328-10011LF, J2 Qwiic_Vertical, J3 679305124022, J4 Qwiic_Vertical, J5 M20-7830542, J6 Qwiic_Vertical, J7 5013310607, J8 Qwiic_4pin_Vertical, J9 Qwiic_Vertical, Q1 BSS138, Q2 BSS138, U1 AP2112K-3.3, U2 BME280, U3 INA219BxDCN, U5 BME280

Commit message: final dreamV3
Connections:
- net GPIO14/TXD0: no longer J6.3 (Pin_3)
- net GPIO15/RXD0: no longer J6.4 (Pin_4)
- net ID_SCL renamed PI9/TXD1
- net PI9/TXD1: now also J6.3 (Pin_3)
- net ID_SDA renamed PI10/RXD1
- net PI10/RXD1: now also J6.4 (Pin_4)

Commit message: Updated PCB
Connections:
- net +3V3: no longer J6.2 (Pin_2)
- net +5V: now also J6.2 (Pin_2)
Changed lines of the file:
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@@
 			)
 		)
-		(property "Value" "+3V3"
+		(property "Value" "+5V"
 			(at 203.2 21.59 90)
 			(show_name no)

Commit message: ACTUAL final DreamV3
Parts:
- IC1: footprint TGS2611_clean:TGS2611C00 -> tgs2611:tgs2611c00; Manufacturer_Part_Number TGS2611-C00 -> SR-6 Sensor Socket; Vendor (none) -> https://www.figarosensor.com/product/entry/sr6.html
- Q2: footprint SparkFun-Semiconductor-Standard:SOT-363 -> PCM_SparkFun-Semiconductor-Standard:SOT-363
- R3: value 10k -> 2k; Vendor https://www.digikey.com/en/products/detail/vishay-dale/CRCW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 -> https://www.digikey.com/en/products/detail/vishay-dale/RCS0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
Connections:
- net GPIO23/SDA4: no longer R5.1
- net GPIO24/SCL4: no longer R5.3
- net GPIO2/SDA1: now also R5.1
- net GPIO3/SCL1: now also R5.3
Other:
- note added: "TGS2611 METHANE SENSOR SOCKET"
- note removed: "TGS2611 METHANE SENSOR"
Changed lines of the file:
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@@
 		)
 	)
-	(text "TGS2611 METHANE SENSOR"
+	(text "TGS2611 METHANE SENSOR SOCKET"
 		(exclude_from_sim no)
-		(at 190.5 122.174 0)
+		(at 194.564 122.174 0)
 		(effects
 			(font
@@
 		)
 	)
-	(label "GPIO23{slash}SDA4"
+	(label "GPIO2{slash}SDA1"
 		(at 15.24 119.38 0)
 		(effects
@@
 		)
 	)
-	(label "GPIO24{slash}SCL4"
+	(label "GPIO3{slash}SCL1"
 		(at 30.48 119.38 0)
 		(effects
@@
 			)
 		)
-		(property "Footprint" "SparkFun-Semiconductor-Standard:SOT-363"
+		(property "Footprint" "PCM_SparkFun-Semiconductor-Standard:SOT-363"
 			(at 151.13 69.85 0)
 			(hide yes)
@@
 			)
 		)
-		(property "Footprint" "SparkFun-Semiconductor-Standard:SOT-363"
+		(property "Footprint" "PCM_SparkFun-Semiconductor-Standard:SOT-363"
 			(at 135.89 83.82 0)
 			(hide yes)
@@
 			)
 		)
-		(property "Footprint" "TGS2611_clean:TGS2611C00"
+		(property "Footprint" "tgs2611:tgs2611c00"
 			(at 256.54 207.95 0)
 			(hide yes)
@@
 			)
 		)
-		(property "Datasheet" "http://www.figarosensor.com/products/docs/TGS%202611C00%281013%29.pdf"
+		(property "Datasheet" "https://www.figarosensor.com/product/sr-6_product%20information%28fusa%29_rev03.pdf"
 			(at 256.54 307.95 0)
 			(hide yes)
@@
 			)
 		)
-		(property "Manufacturer_Part_Number" "TGS2611-C00"
+		(property "Manufacturer_Part_Number" "SR-6 Sensor Socket"
 			(at 256.54 707.95 0)
 			(hide yes)
@@
 			)
 		)
-		(property "Mouser Part Number" ""
-			(at 256.54 807.95 0)
-			(hide yes)
-			(show_name no)
-			(do_not_autoplace no)
-			(effects
-				(font
-					(size 1.27 1.27)
-				)
-				(justify left top)
-			)
-		)
-		(property "Mouser Price/Stock" ""
-			(at 256.54 907.95 0)
-			(hide yes)
-			(show_name no)
-			(do_not_autoplace no)
-			(effects
-				(font
-					(size 1.27 1.27)
-				)
-				(justify left top)
-			)
-		)
-		(property "Arrow Part Number" ""
-			(at 256.54 1007.95 0)
-			(hide yes)
-			(show_name no)
-			(do_not_autoplace no)
-			(effects
-				(font
-					(size 1.27 1.27)
-				)
-				(justify left top)
-			)
-		)
-		(property "Arrow Price/Stock" ""
-			(at 256.54 1107.95 0)
-			(hide yes)
-			(show_name no)
-			(do_not_autoplace no)
-			(effects
-				(font
-					(size 1.27 1.27)
-				)
-				(justify left top)
-			)
-		)
-		(property "Custom Feild" ""
+		(property "Vendor" "https://www.figarosensor.com/product/entry/sr6.html"
 			(at 191.77 113.03 0)
 			(hide yes)
@@
 			)
 		)
-		(property "Value" "10k"
+		(property "Value" "2k"
 			(at 256.54 97.79 0)
 			(show_name no)
@@
 			)
 		)
-		(property "Datasheet" "https://www.vishay.com/docs/20035/dcrcwe3.pdf"
+		(property "Datasheet" "https://www.vishay.com/docs/20065/rcse3.pdf"
 			(at 256.54 91.44 0)
 			(hide yes)
@@
 			)
 		)
-		(property "Vendor" "https://www.digikey.com/en/products/detail/vishay-dale/CRCW060310K0FKEA/1174782"
+		(property "Vendor" "https://www.digikey.com/en/products/detail/vishay-dale/RCS06032K00FKEA/5866936"
 			(at 256.54 100.33 0)
 			(hide yes)

Commit message: ACTUAL final dreamV3
Parts:
- C2: Custom Feild https://www.digikey.com/en/products/detail/taiyo-yuden/TMK2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 -> (none); Vendor (none) -> https://www.digikey.com/en/products/detail/taiyo-yuden/TMK2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
- J1: Vendor (none) -> https://www.digikey.com/en/products/detail/samtec-inc/SSW-1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
- R1, R13: Custom Feild https://www.digikey.com/en/products/detail/bourns-inc/CAT16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 -> (none); Vendor (none) -> https://www.digikey.com/en/products/detail/bourns-inc/CAT16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
- R2, R5: Vendor (none) -> https://www.digikey.com/en/products/detail/bourns-inc/CAT16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
- U1: Custom Feild https://www.digikey.com/en/products/detail/diodes-incorpora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 -> (none); Vendor (none) -> https://www.digikey.com/en/products/detail/diodes-incorpora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
- U2, U5: Vendor (none) -> https://www.digikey.com/en/products/detail/bosch-sensortec/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
- U3: Vendor (none) -> https://www.digikey.com/en/products/detail/texas-instrument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
- renumbered R4 to 0.1
Other:
- note added: "Regulator - Power Safety"
- moved on the sheet: C2
